Commit message: changed 'mecanum' wheel colour to make sure correct robot was loading. Confirmed that mecanum robot is not actually mecanum

File: linorobot2_description/urdf/mech/mecanum_wheel.urdf.xacro (robot description, xacro)
@@ -8,6 +8,6 @@
           <cylinder radius="${radius}" length="${width}"/>
         </geometry>
-        <material name="blue">
-            <color rgba="0.1764 0.4588 0.8509 1.0"/>
+        <material name="red">
+            <color rgba="0.8764 0.4588 0.8509 1.0"/>
         </material>
       </visual>
@@ -33,7 +33,7 @@
       <visual>
         <material>
-          <ambient>0.1764 0.4588 0.8509 1.0</ambient>
-          <diffuse>0.1764 0.4588 0.8509 1.0</diffuse>
-          <specular>0.1764 0.4588 0.8509 1.0</specular>
+          <ambient>0.8764 0.4588 0.8509 1.0</ambient>
+          <diffuse>0.8764 0.4588 0.8509 1.0</diffuse>
+          <specular>0.8764 0.4588 0.8509 1.0</specular>
           <emissive>0.0 0.0 0.0 0.0</emissive>
         </material>

Commit message: Got front left mecanum wheel attach to linorobot2

File: linorobot2_description/urdf/mech/mecanum_wheel.urdf.xacro (robot description, xacro)
@@ -2,47 +2,949 @@
 <robot xmlns:xacro="http://ros.org/wiki/xacro">
   <xacro:macro name="mecanum_wheel" params="side radius width pos_x pos_y pos_z mass">
-    <link name="${side}_wheel_link">
-      <visual>
-        <origin xyz="0 0 0" rpy="${pi/2} 0 0"/>
-        <geometry>
-          <cylinder radius="${radius}" length="${width}"/>
-        </geometry>
-        <material name="red">
-            <color rgba="0.8764 0.4588 0.8509 1.0"/>
-        </material>
-      </visual>
-      <collision>
-        <origin xyz="0 0 0" rpy="${pi/2} 0 0"/>
-        <geometry>
-          <cylinder radius="${radius}" length="${width}"/>
-        </geometry>
-      </collision>
-      <inertial>
-        <origin xyz="0 0 0" rpy="0 0 0"/>
-        <mass value="${mass}"/>
-        <inertia ixx="${(2/5) * mass * (radius * radius)}" ixy="0" ixz="0"
-                 iyy="${(2/5) * mass * (radius * radius)}" iyz="0"
-                 izz="${(2/5) * mass * (radius * radius)}" />
-      </inertial>
-    </link>
-    <gazebo reference="${side}_wheel_link">
-        <mu1>0.01</mu1>
-        <mu2>0.01</mu2>
-    </gazebo>
-    <gazebo reference="${side}_wheel_link">
-      <visual>
-        <material>
-          <ambient>0.8764 0.4588 0.8509 1.0</ambient>
-          <diffuse>0.8764 0.4588 0.8509 1.0</diffuse>
-          <specular>0.8764 0.4588 0.8509 1.0</specular>
-          <emissive>0.0 0.0 0.0 0.0</emissive>
-        </material>
-      </visual>
-    </gazebo>
-    <joint name="${side}_wheel_joint" type="continuous">
-      <axis xyz="0 1 0" />
-      <parent link="base_link"/>
-      <child link="${side}_wheel_link"/>
-      <origin xyz="${pos_x} ${pos_y} ${pos_z}" rpy="0 0 0"/>
+    <link name="${side}_base_link">
+      <inertial>
+        <origin
+          xyz="-3.9077136779291E-16 -0.0136205707454137 -1.44489682185117E-14"
+          rpy="0 0 0" />
+        <mass
+          value="0.039620820516108" />
+        <inertia
+          ixx="3.76577202480009E-05"
+          ixy="-1.07908308681007E-19"
+          ixz="3.89356499633093E-22"
+          iyy="7.10123305553507E-05"
+          iyz="-1.66085499471637E-18"
+          izz="3.76577202480009E-05" />
+      </inertial>
+      <visual>
+        <origin
+          xyz="0 0 0"
+          rpy="0 0 0" />
+        <geometry>
+          <mesh
+            filename="package://linorobot2_description/mecanum_wheel_left/meshes/base_link.STL" />
+        </geometry>
+        <material
+          name="">
+          <color
+            rgba="0.898039215686275 0.917647058823529 0.929411764705882 1" />
+        </material>
+      </visual>
+      <collision>
+        <origin
+          xyz="0 0 0"
+          rpy="0 0 0" />
+        <geometry>
+          <mesh
+            filename="package://linorobot2_description/mecanum_wheel_left/meshes/base_link.STL" />
+        </geometry>
+      </collision>
+    </link>
+    <joint name="base_link_to_${side}_base_link" type="fixed">
+      <origin xyz="${pos_x} ${pos_y} 0"  rpy="0 0 0" />
+      <parent link="base_link" />
+      <child link="${side}_base_link" />
+      <axis xyz="0 0 0" />
+    </joint>
+    <link
+      name="${side}_plate1">
+      <inertial>
+        <origin
+          xyz="8.83119736279022E-16 3.33301269118141E-17 -0.000551568670724527"
+          rpy="0 0 0" />
+        <mass
+          value="0.0253986639693882" />
+        <inertia
+          ixx="4.21627753206923E-05"
+          ixy="1.3976043629696E-20"
+          ixz="-2.39458839321443E-21"
+          iyy="4.21627753206922E-05"
+          iyz="4.06169630282727E-21"
+          izz="8.39719993847474E-05" />
+      </inertial>
+      <visual>
+        <origin
+          xyz="0 0 0"
+          rpy="0 0 0" />
+        <geometry>
+          <mesh
+            filename="package://linorobot2_description/mecanum_wheel_left/meshes/plate1.STL" />
+        </geometry>
+        <material
+          name="">
+          <color
+            rgba="0.650980392156863 0.619607843137255 0.588235294117647 1" />
+        </material>
+      </visual>
+      <collision>
+        <origin
+          xyz="0 0 0"
+          rpy="0 0 0" />
+        <geometry>
+          <mesh
+            filename="package://linorobot2_description/mecanum_wheel_left/meshes/plate1.STL" />
+        </geometry>
+      </collision>
+    </link>
+    <joint
+      name="${side}_base_link_to_${side}_plate1"
+      type="fixed">
+      <origin
+        xyz="0 0.023114 0"
+        rpy="-1.5708 0.03287 0" />
+      <parent
+        link="${side}_base_link" />
+      <child
+        link="${side}_plate1" />
+      <axis
+        xyz="0 0 0" />
+    </joint>
+    <link
+      name="${side}_plate2">
+      <inertial>
+        <origin
+          xyz="-1.10651810076925E-15 8.09386876632109E-17 -0.000551568670724527"
+          rpy="0 0 0" />
+        <mass
+          value="0.0253986639693882" />
+        <inertia
+          ixx="4.21627753206924E-05"
+          ixy="1.65171424714589E-20"
+          ixz="4.28643950323039E-22"
+          iyy="4.21627753206923E-05"
+          iyz="2.75305456980319E-21"
+          izz="8.39719993847476E-05" />
+      </inertial>
+      <visual>
+        <origin
+          xyz="0 0 0"
+          rpy="0 0 0" />
+        <geometry>
+          <mesh
+            filename="package://linorobot2_description/mecanum_wheel_left/meshes/plate2.STL" />
+        </geometry>
+        <material
+          name="">
+          <color
+            rgba="0.650980392156863 0.619607843137255 0.588235294117647 1" />
+        </material>
+      </visual>
+      <collision>
+        <origin
+          xyz="0 0 0"
+          rpy="0 0 0" />
+        <geometry>
+          <mesh
+            filename="package://linorobot2_description/mecanum_wheel_left/meshes/plate2.STL" />
+        </geometry>
+      </collision>
+    </link>
+    <joint
+      name="${side}_base_link_to_${side}_plate2"
+      type="fixed">
+      <origin
+        xyz="0 -0.023114 0"
+        rpy="-1.5707963267949 0.0335546833724646 -3.14159265358979" />
+      <parent
+        link="${side}_base_link" />
+      <child
+        link="${side}_plate2" />
+      <axis
+        xyz="0 0 0" />
+    </joint>
+    <link
+      name="${side}_roller1">
+      <inertial>
+        <origin
+          xyz="5.96744875736022E-16 -1.24475083018716E-14 -0.0215899999999933"
+          rpy="0 0 0" />
+        <mass
+          value="0.00499543658848208" />
+        <inertia
+          ixx="8.99919949242919E-07"
+          ixy="3.97046694025453E-23"
+          ixz="9.81863387100444E-22"
+          iyy="8.9991994924288E-07"
+          iyz="-8.0163727523739E-19"
+          izz="3.31951561004127E-07" />
+      </inertial>
+      <visual>
+        <origin
+          xyz="0 0 0"
+          rpy="0 0 0" />
+        <geometry>
+          <mesh
+            filename="package://linorobot2_description/mecanum_wheel_left/meshes/roller1.STL" />
+        </geometry>
+        <material
+          name="">
+          <color
+            rgba="0.752941176470588 0.752941176470588 0.752941176470588 1" />
+        </material>
+      </visual>
+      <collision>
+        <origin
+          xyz="0 0 0"
+          rpy="0 0 0" />
+        <geometry>
+          <mesh
+            filename="package://linorobot2_description/mecanum_wheel_left/meshes/roller1.STL" />
+        </geometry>
+      </collision>
+    </link>
+    <joint
+      name="${side}_base_link_to_${side}_roller1"
+      type="continuous">
+      <origin
+        xyz="-0.064997 -0.01515 0.019737"
+        rpy="2.3375 0.48899 -0.038445" />
+      <parent
+        link="${side}_base_link" />
+      <child
+        link="${side}_roller1" />
+      <axis
+        xyz="0 0 1" />
+    </joint>
+    <link
+      name="${side}_roller2">
+      <inertial>
+        <origin
+          xyz="5.82867087928207E-16 -9.95687907123788E-15 -0.0215899999999933"
+          rpy="0 0 0" />
+        <mass
+          value="0.00499543658848216" />
+        <inertia
+          ixx="8.99919949245561E-07"
+          ixy="-3.30872245021211E-24"
+          ixz="8.56959114604937E-22"
+          iyy="8.99919949245641E-07"
+          iyz="-8.01716684576195E-19"
+          izz="3.31951561009139E-07" />
+      </inertial>
+      <visual>
+        <origin
+          xyz="0 0 0"
+          rpy="0 0 0" />
+        <geometry>
+          <mesh
+            filename="package://linorobot2_description/mecanum_wheel_left/meshes/roller2.STL" />
+        </geometry>
+        <material
+          name="">
+          <color
+            rgba="0.752941176470588 0.752941176470588 0.752941176470588 1" />
+        </material>
+      </visual>
+      <collision>
+        <origin
+          xyz="0 0 0"
+          rpy="0 0 0" />
+        <geometry>
+          <mesh
+            filename="package://linorobot2_description/mecanum_wheel_left/meshes/roller2.STL" />
+        </geometry>
+      </collision>
+    </link>
+    <joint
+      name="${side}_base_link_to_${side}_roller2"
+      type="continuous">
+      <origin
+        xyz="-0.05135 -0.01515 0.044467"
+        rpy="2.3122 0.90744 -0.055132" />
+      <parent
+        link="${side}_base_link" />
+      <child
+        link="${side}_roller2" />
+      <axis
+        xyz="0 0 1" />
+    </joint>
+    <link
+      name="${side}_roller3">
+      <inertial>
+        <origin
+          xyz="5.82867087928207E-16 -3.41003267290141E-15 -0.0215899999999933"
+          rpy="0 0 0" />
+        <mass
+          value="0.00499543658848228" />
+        <inertia
+          ixx="8.9991994924907E-07"
+          ixy="-9.92616735063633E-24"
+          ixz="8.47860127866853E-22"
+          iyy="8.99919949249046E-07"
+          iyz="-8.01743154355797E-19"
+          izz="3.3195156101569E-07" />
+      </inertial>
+      <visual>
+        <origin
+          xyz="0 0 0"
+          rpy="0 0 0" />
+        <geometry>
+          <mesh
+            filename="package://linorobot2_description/mecanum_wheel_left/meshes/roller3.STL" />
+        </geometry>
+        <material
+          name="">
+          <color
+            rgba="0.752941176470588 0.752941176470588 0.752941176470588 1" />
+        </material>
+      </visual>
+      <collision>
+        <origin
+          xyz="0 0 0"
+          rpy="0 0 0" />
+        <geometry>
+          <mesh
+            filename="package://linorobot2_description/mecanum_wheel_left/meshes/roller3.STL" />
+        </geometry>
+      </collision>
+    </link>
+    <joint
+      name="${side}_base_link_to_${side}_roller3"
+      type="continuous">
+      <origin
+        xyz="-0.028824 -0.01515 0.061508"
+        rpy="2.22 1.3248 -0.13976" />
+      <parent
+        link="${side}_base_link" />
+      <child
+        link="${side}_roller3" />
+      <axis
+        xyz="0 0 1" />
+    </joint>
+    <link
+      name="${side}_roller4">
+      <inertial>
+        <origin
+          xyz="5.68989300120393E-16 -3.35365415993216E-15 -0.0215899999999933"
+          rpy="0 0 0" />
+        <mass
+          value="0.00499543658848229" />
+        <inertia
+          ixx="8.9991994924904E-07"
+          ixy="1.65436122510606E-23"
+          ixz="7.69277969674316E-22"
+          iyy="8.99919949249123E-07"
+          iyz="-8.01796093915E-19"
+          izz="3.31951561015737E-07" />
+      </inertial>
+      <visual>
+        <origin
+          xyz="0 0 0"
+          rpy="0 0 0" />
+        <geometry>
+          <mesh
+            filename="package://linorobot2_description/mecanum_wheel_left/meshes/roller4.STL" />
+        </geometry>
+        <material
+          name="">
+          <color
+            rgba="0.752941176470588 0.752941176470588 0.752941176470588 1" />
+        </material>
+      </visual>
+      <collision>
+        <origin
+          xyz="0 0 0"
+          rpy="0 0 0" />
+        <geometry>
+          <mesh
+            filename="package://linorobot2_description/mecanum_wheel_left/meshes/roller4.STL" />
+        </geometry>
+      </collision>
+    </link>
+    <joint
+      name="${side}_base_link_to_${side}_roller4"
+      type="continuous">
+      <origin
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
File: linorobot2_description/urdf/robots/mecanum.urdf.xacro (robot description, xacro)
@@ -25,5 +25,5 @@
     mass="${wheel_mass}"
   />
-  <xacro:mecanum_wheel
+  <!-- <xacro:mecanum_wheel
     side="front_right"
     radius="${wheel_radius}"
@@ -51,5 +51,5 @@
     pos_z="${wheel_pos_z}"
     mass="${wheel_mass}"
-  />
+  /> -->
   <xacro:imu/>
   <xacro:generic_laser>
