Commit message: Front left and back right mecanum wheels mounted

File: linorobot2_description/urdf/mech/mecanum_wheel.urdf.xacro (robot description, xacro)
@@ -1,6 +1,6 @@
 <?xml version="1.0"?>
 <robot xmlns:xacro="http://ros.org/wiki/xacro">
-  <xacro:macro name="mecanum_wheel" params="side radius width pos_x pos_y pos_z mass">
-    <link name="${side}_base_link">
+  <xacro:macro name="mecanum_wheel" params="mecanum_style end radius width pos_x pos_y pos_z mass">
+    <link name="${end}_${mecanum_style}_base_link">
       <inertial>
         <origin
@@ -23,5 +23,5 @@
         <geometry>
           <mesh
-            filename="package://linorobot2_description/mecanum_wheel_left/meshes/base_link.STL" />
+            filename="package://linorobot2_description/mecanum_wheel_${mecanum_style}/meshes/base_link.STL" />
         </geometry>
         <material
@@ -37,16 +37,16 @@
         <geometry>
           <mesh
-            filename="package://linorobot2_description/mecanum_wheel_left/meshes/base_link.STL" />
-        </geometry>
-      </collision>
-    </link>
-    <joint name="base_link_to_${side}_base_link" type="fixed">
+            filename="package://linorobot2_description/mecanum_wheel_${mecanum_style}/meshes/base_link.STL" />
+        </geometry>
+      </collision>
+    </link>
+    <joint name="base_link_to_${end}_${mecanum_style}_base_link" type="fixed">
       <origin xyz="${pos_x} ${pos_y} 0"  rpy="0 0 0" />
       <parent link="base_link" />
-      <child link="${side}_base_link" />
+      <child link="${end}_${mecanum_style}_base_link" />
       <axis xyz="0 0 0" />
     </joint>
     <link
-      name="${side}_plate1">
+      name="${end}_${mecanum_style}_plate1">
       <inertial>
         <origin
@@ -69,5 +69,5 @@
         <geometry>
           <mesh
-            filename="package://linorobot2_description/mecanum_wheel_left/meshes/plate1.STL" />
+            filename="package://linorobot2_description/mecanum_wheel_${mecanum_style}/meshes/plate1.STL" />
         </geometry>
         <material
@@ -83,10 +83,10 @@
         <geometry>
           <mesh
-            filename="package://linorobot2_description/mecanum_wheel_left/meshes/plate1.STL" />
-        </geometry>
-      </collision>
-    </link>
-    <joint
-      name="${side}_base_link_to_${side}_plate1"
+            filename="package://linorobot2_description/mecanum_wheel_${mecanum_style}/meshes/plate1.STL" />
+        </geometry>
+      </collision>
+    </link>
+    <joint
+      name="${end}_${mecanum_style}_base_link_to_${end}_${mecanum_style}_plate1"
       type="fixed">
       <origin
@@ -94,12 +94,12 @@
         rpy="-1.5708 0.03287 0" />
       <parent
-        link="${side}_base_link" />
-      <child
-        link="${side}_plate1" />
+        link="${end}_${mecanum_style}_base_link" />
+      <child
+        link="${end}_${mecanum_style}_plate1" />
       <axis
         xyz="0 0 0" />
     </joint>
     <link
-      name="${side}_plate2">
+      name="${end}_${mecanum_style}_plate2">
       <inertial>
         <origin
@@ -122,5 +122,5 @@
         <geometry>
           <mesh
-            filename="package://linorobot2_description/mecanum_wheel_left/meshes/plate2.STL" />
+            filename="package://linorobot2_description/mecanum_wheel_${mecanum_style}/meshes/plate2.STL" />
         </geometry>
         <material
@@ -136,10 +136,10 @@
         <geometry>
           <mesh
-            filename="package://linorobot2_description/mecanum_wheel_left/meshes/plate2.STL" />
-        </geometry>
-      </collision>
-    </link>
-    <joint
-      name="${side}_base_link_to_${side}_plate2"
+            filename="package://linorobot2_description/mecanum_wheel_${mecanum_style}/meshes/plate2.STL" />
+        </geometry>
+      </collision>
+    </link>
+    <joint
+      name="${end}_${mecanum_style}_base_link_to_${end}_${mecanum_style}_plate2"
       type="fixed">
       <origin
@@ -147,12 +147,12 @@
         rpy="-1.5707963267949 0.0335546833724646 -3.14159265358979" />
       <parent
-        link="${side}_base_link" />
-      <child
-        link="${side}_plate2" />
+        link="${end}_${mecanum_style}_base_link" />
+      <child
+        link="${end}_${mecanum_style}_plate2" />
       <axis
         xyz="0 0 0" />
     </joint>
     <link
-      name="${side}_roller1">
+      name="${end}_${mecanum_style}_roller1">
       <inertial>
         <origin
@@ -175,24 +175,24 @@
         <geometry>
           <mesh
-            filename="package://linorobot2_description/mecanum_wheel_left/meshes/roller1.STL" />
-        </geometry>
-        <material
-          name="">
-          <color
-            rgba="0.752941176470588 0.752941176470588 0.752941176470588 1" />
-        </material>
-      </visual>
-      <collision>
-        <origin
-          xyz="0 0 0"
-          rpy="0 0 0" />
-        <geometry>
-          <mesh
-            filename="package://linorobot2_description/mecanum_wheel_left/meshes/roller1.STL" />
-        </geometry>
-      </collision>
-    </link>
-    <joint
-      name="${side}_base_link_to_${side}_roller1"
+            filename="package://linorobot2_description/mecanum_wheel_${mecanum_style}/meshes/roller1.STL" />
+        </geometry>
+        <material
+          name="">
+          <color
+            rgba="0.752941176470588 0.752941176470588 0.752941176470588 1" />
+        </material>
+      </visual>
+      <collision>
+        <origin
+          xyz="0 0 0"
+          rpy="0 0 0" />
+        <geometry>
+          <mesh
+            filename="package://linorobot2_description/mecanum_wheel_${mecanum_style}/meshes/roller1.STL" />
+        </geometry>
+      </collision>
+    </link>
+    <joint
+      name="${end}_${mecanum_style}_base_link_to_${end}_${mecanum_style}_roller1"
       type="continuous">
       <origin
@@ -200,12 +200,12 @@
         rpy="2.3375 0.48899 -0.038445" />
       <parent
-        link="${side}_base_link" />
-      <child
-        link="${side}_roller1" />
-      <axis
-        xyz="0 0 1" />
-    </joint>
-    <link
-      name="${side}_roller2">
+        link="${end}_${mecanum_style}_base_link" />
+      <child
+        link="${end}_${mecanum_style}_roller1" />
+      <axis
+        xyz="0 0 1" />
+    </joint>
+    <link
+      name="${end}_${mecanum_style}_roller2">
       <inertial>
         <origin
@@ -228,24 +228,24 @@
         <geometry>
           <mesh
-            filename="package://linorobot2_description/mecanum_wheel_left/meshes/roller2.STL" />
-        </geometry>
-        <material
-          name="">
-          <color
-            rgba="0.752941176470588 0.752941176470588 0.752941176470588 1" />
-        </material>
-      </visual>
-      <collision>
-        <origin
-          xyz="0 0 0"
-          rpy="0 0 0" />
-        <geometry>
-          <mesh
-            filename="package://linorobot2_description/mecanum_wheel_left/meshes/roller2.STL" />
-        </geometry>
-      </collision>
-    </link>
-    <joint
-      name="${side}_base_link_to_${side}_roller2"
+            filename="package://linorobot2_description/mecanum_wheel_${mecanum_style}/meshes/roller2.STL" />
+        </geometry>
+        <material
+          name="">
+          <color
+            rgba="0.752941176470588 0.752941176470588 0.752941176470588 1" />
+        </material>
+      </visual>
+      <collision>
+        <origin
+          xyz="0 0 0"
+          rpy="0 0 0" />
+        <geometry>
+          <mesh
+            filename="package://linorobot2_description/mecanum_wheel_${mecanum_style}/meshes/roller2.STL" />
+        </geometry>
+      </collision>
+    </link>
+    <joint
+      name="${end}_${mecanum_style}_base_link_to_${end}_${mecanum_style}_roller2"
       type="continuous">
       <origin
@@ -253,12 +253,12 @@
         rpy="2.3122 0.90744 -0.055132" />
       <parent
-        link="${side}_base_link" />
-      <child
-        link="${side}_roller2" />
-      <axis
-        xyz="0 0 1" />
-    </joint>
-    <link
-      name="${side}_roller3">
+        link="${end}_${mecanum_style}_base_link" />
+      <child
+        link="${end}_${mecanum_style}_roller2" />
+      <axis
+        xyz="0 0 1" />
+    </joint>
+    <link
+      name="${end}_${mecanum_style}_roller3">
       <inertial>
         <origin
@@ -281,24 +281,24 @@
         <geometry>
           <mesh
-            filename="package://linorobot2_description/mecanum_wheel_left/meshes/roller3.STL" />
-        </geometry>
-        <material
-          name="">
-          <color
-            rgba="0.752941176470588 0.752941176470588 0.752941176470588 1" />
-        </material>
-      </visual>
-      <collision>
-        <origin
-          xyz="0 0 0"
-          rpy="0 0 0" />
-        <geometry>
-          <mesh
-            filename="package://linorobot2_description/mecanum_wheel_left/meshes/roller3.STL" />
-        </geometry>
-      </collision>
-    </link>
-    <joint
-      name="${side}_base_link_to_${side}_roller3"
+            filename="package://linorobot2_description/mecanum_wheel_${mecanum_style}/meshes/roller3.STL" />
+        </geometry>
+        <material
+          name="">
+          <color
+            rgba="0.752941176470588 0.752941176470588 0.752941176470588 1" />
+        </material>
+      </visual>
+      <collision>
+        <origin
+          xyz="0 0 0"
+          rpy="0 0 0" />
+        <geometry>
+          <mesh
+            filename="package://linorobot2_description/mecanum_wheel_${mecanum_style}/meshes/roller3.STL" />
+        </geometry>
+      </collision>
+    </link>
+    <joint
+      name="${end}_${mecanum_style}_base_link_to_${end}_${mecanum_style}_roller3"
       type="continuous">
       <origin
@@ -306,12 +306,12 @@
         rpy="2.22 1.3248 -0.13976" />
       <parent
-        link="${side}_base_link" />
-      <child
-        link="${side}_roller3" />
-      <axis
-        xyz="0 0 1" />
-    </joint>
-    <link
-      name="${side}_roller4">
+        link="${end}_${mecanum_style}_base_link" />
+      <child
+        link="${end}_${mecanum_style}_roller3" />
+      <axis
+        xyz="0 0 1" />
+    </joint>
+    <link
+      name="${end}_${mecanum_style}_roller4">
       <inertial>
         <origin
@@ -334,24 +334,24 @@
         <geometry>
           <mesh
-            filename="package://linorobot2_description/mecanum_wheel_left/meshes/roller4.STL" />
-        </geometry>
-        <material
-          name="">
-          <color
-            rgba="0.752941176470588 0.752941176470588 0.752941176470588 1" />
-        </material>
-      </visual>
-      <collision>
-        <origin
-          xyz="0 0 0"
-          rpy="0 0 0" />
-        <geometry>
-          <mesh
-            filename="package://linorobot2_description/mecanum_wheel_left/meshes/roller4.STL" />
-        </geometry>
-      </collision>
-    </link>
-    <joint
-      name="${side}_base_link_to_${side}_roller4"
+            filename="package://linorobot2_description/mecanum_wheel_${mecanum_style}/meshes/roller4.STL" />
+        </geometry>
+        <material
+          name="">
+          <color
+            rgba="0.752941176470588 0.752941176470588 0.752941176470588 1" />
+        </material>
+      </visual>
+      <collision>
+        <origin
+          xyz="0 0 0"
+          rpy="0 0 0" />
+        <geometry>
+          <mesh
+            filename="package://linorobot2_description/mecanum_wheel_${mecanum_style}/meshes/roller4.STL" />
+        </geometry>
+      </collision>
+    </link>
+    <joint
+      name="${end}_${mecanum_style}_base_link_to_${end}_${mecanum_style}_roller4"
       type="continuous">
       <origin
@@ -359,12 +359,12 @@
         rpy="-0.59653 1.3924 -2.9492" />
       <parent
-        link="${side}_base_link" />
-      <child
-        link="${side}_roller4" />
-      <axis
-        xyz="0 0 1" />
-    </joint>
-    <link
-      name="${side}_roller5">
+        link="${end}_${mecanum_style}_base_link" />
+      <child
+        link="${end}_${mecanum_style}_roller4" />
+      <axis
+        xyz="0 0 1" />
+    </joint>
+    <link
+      name="${end}_${mecanum_style}_roller5">
       <inertial>
         <origin
@@ -387,24 +387,24 @@
         <geometry>
           <mesh
-            filename="package://linorobot2_description/mecanum_wheel_left/meshes/roller5.STL" />
-        </geometry>
-        <material
-          name="">
-          <color
-            rgba="0.752941176470588 0.752941176470588 0.752941176470588 1" />
-        </material>
-      </visual>
-      <collision>
-        <origin
-          xyz="0 0 0"
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
File: linorobot2_description/urdf/robots/mecanum.urdf.xacro (robot description, xacro)
@@ -17,5 +17,6 @@
 />
   <xacro:mecanum_wheel
-    side="front_left"
+    mecanum_style="left"
+    end="front"
     radius="${wheel_radius}"
     width="${wheel_width}"
@@ -26,5 +27,5 @@
   />
   <!-- <xacro:mecanum_wheel
-    side="front_right"
+    mecanum_style="front_right"
     radius="${wheel_radius}"
     width="${wheel_width}"
@@ -33,7 +34,8 @@
     pos_z="${wheel_pos_z}"
     mass="${wheel_mass}"
-  />
-  <xacro:mecanum_wheel
-    side="rear_left"
+  /> -->
+  <!-- <xacro:mecanum_wheel
+    mecanum_style="left"
+    end="rear"
     radius="${wheel_radius}"
     width="${wheel_width}"
@@ -42,7 +44,9 @@
     pos_z="${wheel_pos_z}"
     mass="${wheel_mass}"
-  />
+  /> -->
+  <!-- Left style mecanum wheel is on back RIGHT of robot -->
   <xacro:mecanum_wheel
-    side="rear_right"
+    mecanum_style="left"
+    end="rear"
     radius="${wheel_radius}"
     width="${wheel_width}"
@@ -51,5 +55,5 @@
     pos_z="${wheel_pos_z}"
     mass="${wheel_mass}"
-  /> -->
+  />
   <xacro:imu/>
   <xacro:generic_laser>
