Commit message: Got linorobot with 1 mecanum wheel loaded into isaacsim

File: linorobot2_description/urdf/mech/base.urdf.xacro (robot description, xacro)
@@ -28,14 +28,4 @@
       </inertial>
     </link>
-    <gazebo reference="base_link">
-      <visual>
-        <material>
-          <ambient>0.8392 0.6314 0.0 1.0</ambient>
-          <diffuse>0.8392 0.6314 0.0 1.0</diffuse>
-          <specular>0.99 0.99 0.99 1.0</specular>
-          <emissive>0.0 0.0 0.0 0.0</emissive>
-        </material>
-      </visual>
-    </gazebo>
     <joint name="base_to_footprint" type="fixed">
       <parent link="base_footprint"/>

File: linorobot2_description/urdf/mech/mecanum_wheel_left.urdf.xacro (robot description, xacro)
@@ -23,5 +23,5 @@
         <geometry>
           <mesh
-            filename="package://linorobot2_description/mecanum_wheel_left/meshes/base_link.STL" />
+            filename="package://linorobot2_description/meshes/mecanum_wheel_left/base_link.STL" />
         </geometry>
         <material
@@ -37,5 +37,5 @@
         <geometry>
           <mesh
-            filename="package://linorobot2_description/mecanum_wheel_left/meshes/base_link.STL" />
+            filename="package://linorobot2_description/meshes/mecanum_wheel_left/base_link.STL" />
         </geometry>
       </collision>
@@ -69,5 +69,5 @@
         <geometry>
           <mesh
-            filename="package://linorobot2_description/mecanum_wheel_left/meshes/plate1.STL" />
+            filename="package://linorobot2_description/meshes/mecanum_wheel_left/plate1.STL" />
         </geometry>
         <material
@@ -83,5 +83,5 @@
         <geometry>
           <mesh
-            filename="package://linorobot2_description/mecanum_wheel_left/meshes/plate1.STL" />
+            filename="package://linorobot2_description/meshes/mecanum_wheel_left/plate1.STL" />
         </geometry>
       </collision>
@@ -122,5 +122,5 @@
         <geometry>
           <mesh
-            filename="package://linorobot2_description/mecanum_wheel_left/meshes/plate2.STL" />
+            filename="package://linorobot2_description/meshes/mecanum_wheel_left/plate2.STL" />
         </geometry>
         <material
@@ -136,5 +136,5 @@
         <geometry>
           <mesh
-            filename="package://linorobot2_description/mecanum_wheel_left/meshes/plate2.STL" />
+            filename="package://linorobot2_description/meshes/mecanum_wheel_left/plate2.STL" />
         </geometry>
       </collision>
@@ -175,19 +175,19 @@
         <geometry>
           <mesh
-            filename="package://linorobot2_description/mecanum_wheel_left/meshes/roller1.STL" />
-        </geometry>
-        <material
-          name="">
-          <color
-            rgba="0.752941176470588 0.752941176470588 0.752941176470588 1" />
-        </material>
-      </visual>
-      <collision>
-        <origin
-          xyz="0 0 0"
-          rpy="0 0 0" />
-        <geometry>
-          <mesh
-            filename="package://linorobot2_description/mecanum_wheel_left/meshes/roller1.STL" />
+            filename="package://linorobot2_description/meshes/mecanum_wheel_left/roller1.STL" />
+        </geometry>
+        <material
+          name="">
+          <color
+            rgba="0.752941176470588 0.752941176470588 0.752941176470588 1" />
+        </material>
+      </visual>
+      <collision>
+        <origin
+          xyz="0 0 0"
+          rpy="0 0 0" />
+        <geometry>
+          <mesh
+            filename="package://linorobot2_description/meshes/mecanum_wheel_left/roller1.STL" />
         </geometry>
       </collision>
@@ -228,19 +228,19 @@
         <geometry>
           <mesh
-            filename="package://linorobot2_description/mecanum_wheel_left/meshes/roller2.STL" />
-        </geometry>
-        <material
-          name="">
-          <color
-            rgba="0.752941176470588 0.752941176470588 0.752941176470588 1" />
-        </material>
-      </visual>
-      <collision>
-        <origin
-          xyz="0 0 0"
-          rpy="0 0 0" />
-        <geometry>
-          <mesh
-            filename="package://linorobot2_description/mecanum_wheel_left/meshes/roller2.STL" />
+            filename="package://linorobot2_description/meshes/mecanum_wheel_left/roller2.STL" />
+        </geometry>
+        <material
+          name="">
+          <color
+            rgba="0.752941176470588 0.752941176470588 0.752941176470588 1" />
+        </material>
+      </visual>
+      <collision>
+        <origin
+          xyz="0 0 0"
+          rpy="0 0 0" />
+        <geometry>
+          <mesh
+            filename="package://linorobot2_description/meshes/mecanum_wheel_left/roller2.STL" />
         </geometry>
       </collision>
@@ -281,19 +281,19 @@
         <geometry>
           <mesh
-            filename="package://linorobot2_description/mecanum_wheel_left/meshes/roller3.STL" />
-        </geometry>
-        <material
-          name="">
-          <color
-            rgba="0.752941176470588 0.752941176470588 0.752941176470588 1" />
-        </material>
-      </visual>
-      <collision>
-        <origin
-          xyz="0 0 0"
-          rpy="0 0 0" />
-        <geometry>
-          <mesh
-            filename="package://linorobot2_description/mecanum_wheel_left/meshes/roller3.STL" />
+            filename="package://linorobot2_description/meshes/mecanum_wheel_left/roller3.STL" />
+        </geometry>
+        <material
+          name="">
+          <color
+            rgba="0.752941176470588 0.752941176470588 0.752941176470588 1" />
+        </material>
+      </visual>
+      <collision>
+        <origin
+          xyz="0 0 0"
+          rpy="0 0 0" />
+        <geometry>
+          <mesh
+            filename="package://linorobot2_description/meshes/mecanum_wheel_left/roller3.STL" />
         </geometry>
       </collision>
@@ -334,19 +334,19 @@
         <geometry>
           <mesh
-            filename="package://linorobot2_description/mecanum_wheel_left/meshes/roller4.STL" />
-        </geometry>
-        <material
-          name="">
-          <color
-            rgba="0.752941176470588 0.752941176470588 0.752941176470588 1" />
-        </material>
-      </visual>
-      <collision>
-        <origin
-          xyz="0 0 0"
-          rpy="0 0 0" />
-        <geometry>
-          <mesh
-            filename="package://linorobot2_description/mecanum_wheel_left/meshes/roller4.STL" />
+            filename="package://linorobot2_description/meshes/mecanum_wheel_left/roller4.STL" />
+        </geometry>
+        <material
+          name="">
+          <color
+            rgba="0.752941176470588 0.752941176470588 0.752941176470588 1" />
+        </material>
+      </visual>
+      <collision>
+        <origin
+          xyz="0 0 0"
+          rpy="0 0 0" />
+        <geometry>
+          <mesh
+            filename="package://linorobot2_description/meshes/mecanum_wheel_left/roller4.STL" />
         </geometry>
       </collision>
@@ -387,19 +387,19 @@
         <geometry>
           <mesh
-            filename="package://linorobot2_description/mecanum_wheel_left/meshes/roller5.STL" />
-        </geometry>
-        <material
-          name="">
-          <color
-            rgba="0.752941176470588 0.752941176470588 0.752941176470588 1" />
-        </material>
-      </visual>
-      <collision>
-        <origin
-          xyz="0 0 0"
-          rpy="0 0 0" />
-        <geometry>
-          <mesh
-            filename="package://linorobot2_description/mecanum_wheel_left/meshes/roller5.STL" />
+            filename="package://linorobot2_description/meshes/mecanum_wheel_left/roller5.STL" />
+        </geometry>
+        <material
+          name="">
+          <color
+            rgba="0.752941176470588 0.752941176470588 0.752941176470588 1" />
+        </material>
+      </visual>
+      <collision>
+        <origin
+          xyz="0 0 0"
+          rpy="0 0 0" />
+        <geometry>
+          <mesh
+            filename="package://linorobot2_description/meshes/mecanum_wheel_left/roller5.STL" />
         </geometry>
       </collision>
@@ -440,19 +440,19 @@
         <geometry>
           <mesh
-            filename="package://linorobot2_description/mecanum_wheel_left/meshes/roller6.STL" />
-        </geometry>
-        <material
-          name="">
-          <color
-            rgba="0.752941176470588 0.752941176470588 0.752941176470588 1" />
-        </material>
-      </visual>
-      <collision>
-        <origin
-          xyz="0 0 0"
-          rpy="0 0 0" />
-        <geometry>
-          <mesh
-            filename="package://linorobot2_description/mecanum_wheel_left/meshes/roller6.STL" />
+            filename="package://linorobot2_description/meshes/mecanum_wheel_left/roller6.STL" />
+        </geometry>
+        <material
+          name="">
+          <color
+            rgba="0.752941176470588 0.752941176470588 0.752941176470588 1" />
+        </material>
+      </visual>
+      <collision>
+        <origin
+          xyz="0 0 0"
+          rpy="0 0 0" />
+        <geometry>
+          <mesh
+            filename="package://linorobot2_description/meshes/mecanum_wheel_left/roller6.STL" />
         </geometry>
       </collision>
@@ -493,19 +493,19 @@
         <geometry>
           <mesh
-            filename="package://linorobot2_description/mecanum_wheel_left/meshes/roller7.STL" />
-        </geometry>
-        <material
-          name="">
-          <color
-            rgba="0.752941176470588 0.752941176470588 0.752941176470588 1" />
-        </material>
-      </visual>
-      <collision>
-        <origin
-          xyz="0 0 0"
-          rpy="0 0 0" />
-        <geometry>
-          <mesh
-            filename="package://linorobot2_description/mecanum_wheel_left/meshes/roller7.STL" />
+            filename="package://linorobot2_description/meshes/mecanum_wheel_left/roller7.STL" />
+        </geometry>
+        <material
+          name="">
+          <color
+            rgba="0.752941176470588 0.752941176470588 0.752941176470588 1" />
+        </material>
+      </visual>
+      <collision>
+        <origin
+          xyz="0 0 0"
+          rpy="0 0 0" />
+        <geometry>
+          <mesh
+            filename="package://linorobot2_description/meshes/mecanum_wheel_left/roller7.STL" />
         </geometry>
       </collision>
@@ -546,19 +546,19 @@
         <geometry>
           <mesh
-            filename="package://linorobot2_description/mecanum_wheel_left/meshes/roller8.STL" />
-        </geometry>
-        <material
-          name="">
-          <color
-            rgba="0.752941176470588 0.752941176470588 0.752941176470588 1" />
-        </material>
-      </visual>
-      <collision>
-        <origin
-          xyz="0 0 0"
-          rpy="0 0 0" />
-        <geometry>
-          <mesh
-            filename="package://linorobot2_description/mecanum_wheel_left/meshes/roller8.STL" />
+            filename="package://linorobot2_description/meshes/mecanum_wheel_left/roller8.STL" />
+        </geometry>
+        <material
+          name="">
+          <color
+            rgba="0.752941176470588 0.752941176470588 0.752941176470588 1" />
+        </material>
+      </visual>
+      <collision>
+        <origin
+          xyz="0 0 0"
+          rpy="0 0 0" />
+        <geometry>
+          <mesh
+            filename="package://linorobot2_description/meshes/mecanum_wheel_left/roller8.STL" />
         </geometry>
       </collision>
@@ -599,19 +599,19 @@
         <geometry>
           <mesh
-            filename="package://linorobot2_description/mecanum_wheel_left/meshes/roller9.STL" />
-        </geometry>
-        <material
-          name="">
-          <color
-            rgba="0.752941176470588 0.752941176470588 0.752941176470588 1" />
-        </material>
-      </visual>
-      <collision>
-        <origin
-          xyz="0 0 0"
-          rpy="0 0 0" />
-        <geometry>
-          <mesh
-            filename="package://linorobot2_description/mecanum_wheel_left/meshes/roller9.STL" />
+            filename="package://linorobot2_description/meshes/mecanum_wheel_left/roller9.STL" />
+        </geometry>
+        <material
+          name="">
+          <color
+            rgba="0.752941176470588 0.752941176470588 0.752941176470588 1" />
+        </material>
+      </visual>
+      <collision>
+        <origin
+          xyz="0 0 0"
+          rpy="0 0 0" />
+        <geometry>
+          <mesh
+            filename="package://linorobot2_description/meshes/mecanum_wheel_left/roller9.STL" />
         </geometry>
       </collision>
@@ -652,19 +652,19 @@
         <geometry>
           <mesh
-            filename="package://linorobot2_description/mecanum_wheel_left/meshes/roller10.STL" />
-        </geometry>
-        <material
-          name="">
-          <color
-            rgba="0.752941176470588 0.752941176470588 0.752941176470588 1" />
-        </material>
-      </visual>
-      <collision>
-        <origin
-          xyz="0 0 0"
-          rpy="0 0 0" />
-        <geometry>
-          <mesh
-            filename="package://linorobot2_description/mecanum_wheel_left/meshes/roller10.STL" />
+            filename="package://linorobot2_description/meshes/mecanum_wheel_left/roller10.STL" />
+        </geometry>
+        <material
+          name="">
+          <color
+            rgba="0.752941176470588 0.752941176470588 0.752941176470588 1" />
+        </material>
+      </visual>
+      <collision>
+        <origin
+          xyz="0 0 0"
+          rpy="0 0 0" />
+        <geometry>
+          <mesh
+            filename="package://linorobot2_description/meshes/mecanum_wheel_left/roller10.STL" />
         </geometry>
       </collision>
@@ -705,19 +705,19 @@
         <geometry>
           <mesh
-            filename="package://linorobot2_description/mecanum_wheel_left/meshes/roller11.STL" />
-        </geometry>
-        <material
-          name="">
-          <color
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
File: linorobot2_description/urdf/robots/mecanum.urdf.xacro (robot description, xacro)
@@ -5,8 +5,8 @@
   <xacro:include filename="$(find linorobot2_description)/urdf/mech/mecanum_wheel_left.urdf.xacro" />
   <xacro:include filename="$(find linorobot2_description)/urdf/mech/mecanum_wheel_right.urdf.xacro" />
-  <xacro:include filename="$(find linorobot2_description)/urdf/sensors/imu.urdf.xacro" />
+  <!-- <xacro:include filename="$(find linorobot2_description)/urdf/sensors/imu.urdf.xacro" />
   <xacro:include filename="$(find linorobot2_description)/urdf/sensors/generic_laser.urdf.xacro" />
   <xacro:include filename="$(find linorobot2_description)/urdf/sensors/depth_sensor.urdf.xacro" />
-  <xacro:include filename="$(find linorobot2_description)/urdf/controllers/omni_drive.urdf.xacro" />
+  <xacro:include filename="$(find linorobot2_description)/urdf/controllers/omni_drive.urdf.xacro" /> -->
   <xacro:base
     length="${base_length}"
@@ -27,5 +27,5 @@
     mass="${wheel_mass}"
   />
-  <xacro:mecanum_wheel_right
+  <!-- <xacro:mecanum_wheel_right
     side="right"
     end="front"
@@ -36,7 +36,7 @@
     pos_z="${wheel_pos_z}"
     mass="${wheel_mass}"
-  />
+  /> -->
   <!-- Back wheels mechanum style swapped (left mecanum wheel goes on right side of robot, and vice versa) -->
-  <xacro:mecanum_wheel_right
+  <!-- <xacro:mecanum_wheel_right
     side="left"
     end="rear"
@@ -57,12 +57,4 @@
     pos_z="${wheel_pos_z}"
     mass="${wheel_mass}"
-  />
-  <xacro:imu/>
-  <xacro:generic_laser>
-    <xacro:insert_block name="laser_pose" />
-  </xacro:generic_laser>
-  <xacro:depth_sensor>
-    <xacro:insert_block name="depth_sensor_pose" />
-  </xacro:depth_sensor>
-  <xacro:omni_drive_controller/>
+  /> -->
 </robot>
