Commit message: Added a lot of damping to wheel joints to minimize robot bumpiness

File: linorobot2_description/urdf/mech/base.urdf.xacro (robot description, xacro)
@@ -23,7 +23,4 @@
         <origin xyz="0 0 0" rpy="0 0 0"/>
         <mass value="${mass}"/>
-        <inertia ixx="${(1/12) * mass * ((width  * width)  + (height * height))}" ixy="0.0" ixz="0.0"
-                 iyy="${(1/12) * mass * ((length * length) + (height * height))}" iyz="0.0"
-                 izz="${(1/12) * mass * ((length * length) + (width  * width))}"/>
       </inertial>
     </link>

File: linorobot2_description/urdf/mech/end_channel.urdf.xacro (robot description, xacro)
@@ -16,4 +16,7 @@
         </geometry>
       </collision>
+      <inertial>
+        <mass value="5"/>
+      </inertial>
     </link>
     <joint name="base_link_to_${end}_channel" type="fixed">

File: linorobot2_description/urdf/mech/mecanum_wheel_left.urdf.xacro (robot description, xacro)
@@ -2,5 +2,5 @@
 <robot xmlns:xacro="http://ros.org/wiki/xacro">
   <xacro:macro name="mecanum_wheel_left" params="side end radius width pos_x pos_y pos_z mass">
-    <link name="${end}_${side}_base_link">
+    <link name="${end}_${side}_wheel">
       <inertial>
         <origin
@@ -8,12 +8,5 @@
           rpy="0 0 0" />
         <mass
-          value="0.039620820516108" />
-        <inertia
-          ixx="3.76577202480009E-05"
-          ixy="-1.07908308681007E-19"
-          ixz="3.89356499633093E-22"
-          iyy="7.10123305553507E-05"
-          iyz="-1.66085499471637E-18"
-          izz="3.76577202480009E-05" />
+          value="0.25" />
       </inertial>
       <visual>
@@ -41,8 +34,8 @@
       </collision>
     </link>
-    <joint name="base_link_to_${end}_${side}_base_link" type="continuous">
+    <joint name="base_link_to_${end}_${side}_wheel" type="continuous">
       <origin xyz="${pos_x} ${pos_y} 0"  rpy="0 0 0" />
       <parent link="base_link" />
-      <child link="${end}_${side}_base_link" />
+      <child link="${end}_${side}_wheel" />
       <axis xyz="0 1 0" />
     </joint>
@@ -50,16 +43,6 @@
       name="${end}_${side}_plate1">
       <inertial>
-        <origin
-          xyz="8.83119736279022E-16 3.33301269118141E-17 -0.000551568670724527"
-          rpy="0 0 0" />
-        <mass
-          value="0.0253986639693882" />
-        <inertia
-          ixx="4.21627753206923E-05"
-          ixy="1.3976043629696E-20"
-          ixz="-2.39458839321443E-21"
-          iyy="4.21627753206922E-05"
-          iyz="4.06169630282727E-21"
-          izz="8.39719993847474E-05" />
+        <mass
+          value="0.5" />
       </inertial>
       <visual>
@@ -88,5 +71,5 @@
     </link>
     <joint
-      name="${end}_${side}_base_link_to_${end}_${side}_plate1"
+      name="${end}_${side}_wheel_to_${end}_${side}_plate1"
       type="fixed">
       <origin
@@ -94,5 +77,5 @@
         rpy="-1.5708 0.03287 0" />
       <parent
-        link="${end}_${side}_base_link" />
+        link="${end}_${side}_wheel" />
       <child
         link="${end}_${side}_plate1" />
@@ -103,16 +86,5 @@
       name="${end}_${side}_plate2">
       <inertial>
-        <origin
-          xyz="-1.10651810076925E-15 8.09386876632109E-17 -0.000551568670724527"
-          rpy="0 0 0" />
-        <mass
-          value="0.0253986639693882" />
-        <inertia
-          ixx="4.21627753206924E-05"
-          ixy="1.65171424714589E-20"
-          ixz="4.28643950323039E-22"
-          iyy="4.21627753206923E-05"
-          iyz="2.75305456980319E-21"
-          izz="8.39719993847476E-05" />
+        <mass value="0.5" />
       </inertial>
       <visual>
@@ -141,5 +113,5 @@
     </link>
     <joint
-      name="${end}_${side}_base_link_to_${end}_${side}_plate2"
+      name="${end}_${side}_wheel_to_${end}_${side}_plate2"
       type="fixed">
       <origin
@@ -147,5 +119,5 @@
         rpy="-1.5707963267949 0.0335546833724646 -3.14159265358979" />
       <parent
-        link="${end}_${side}_base_link" />
+        link="${end}_${side}_wheel" />
       <child
         link="${end}_${side}_plate2" />
@@ -160,12 +132,5 @@
           rpy="0 0 0" />
         <mass
-          value="0.00499543658848208" />
-        <inertia
-          ixx="8.99919949242919E-07"
-          ixy="3.97046694025453E-23"
-          ixz="9.81863387100444E-22"
-          iyy="8.9991994924288E-07"
-          iyz="-8.0163727523739E-19"
-          izz="3.31951561004127E-07" />
+          value="0.025" />
       </inertial>
       <visual>
@@ -194,5 +159,5 @@
     </link>
     <joint
-      name="${end}_${side}_base_link_to_${end}_${side}_roller1"
+      name="${end}_${side}_wheel_to_${end}_${side}_roller1"
       type="continuous">
       <origin
@@ -200,5 +165,5 @@
         rpy="2.3375 0.48899 -0.038445" />
       <parent
-        link="${end}_${side}_base_link" />
+        link="${end}_${side}_wheel" />
       <child
         link="${end}_${side}_roller1" />
@@ -213,12 +178,5 @@
           rpy="0 0 0" />
         <mass
-          value="0.00499543658848216" />
-        <inertia
-          ixx="8.99919949245561E-07"
-          ixy="-3.30872245021211E-24"
-          ixz="8.56959114604937E-22"
-          iyy="8.99919949245641E-07"
-          iyz="-8.01716684576195E-19"
-          izz="3.31951561009139E-07" />
+          value="0.025" />
       </inertial>
       <visual>
@@ -247,5 +205,5 @@
     </link>
     <joint
-      name="${end}_${side}_base_link_to_${end}_${side}_roller2"
+      name="${end}_${side}_wheel_to_${end}_${side}_roller2"
       type="continuous">
       <origin
@@ -253,5 +211,5 @@
         rpy="2.3122 0.90744 -0.055132" />
       <parent
-        link="${end}_${side}_base_link" />
+        link="${end}_${side}_wheel" />
       <child
         link="${end}_${side}_roller2" />
@@ -266,12 +224,5 @@
           rpy="0 0 0" />
         <mass
-          value="0.00499543658848228" />
-        <inertia
-          ixx="8.9991994924907E-07"
-          ixy="-9.92616735063633E-24"
-          ixz="8.47860127866853E-22"
-          iyy="8.99919949249046E-07"
-          iyz="-8.01743154355797E-19"
-          izz="3.3195156101569E-07" />
+          value="0.025" />
       </inertial>
       <visual>
@@ -300,5 +251,5 @@
     </link>
     <joint
-      name="${end}_${side}_base_link_to_${end}_${side}_roller3"
+      name="${end}_${side}_wheel_to_${end}_${side}_roller3"
       type="continuous">
       <origin
@@ -306,5 +257,5 @@
         rpy="2.22 1.3248 -0.13976" />
       <parent
-        link="${end}_${side}_base_link" />
+        link="${end}_${side}_wheel" />
       <child
         link="${end}_${side}_roller3" />
@@ -319,12 +270,5 @@
           rpy="0 0 0" />
         <mass
-          value="0.00499543658848229" />
-        <inertia
-          ixx="8.9991994924904E-07"
-          ixy="1.65436122510606E-23"
-          ixz="7.69277969674316E-22"
-          iyy="8.99919949249123E-07"
-          iyz="-8.01796093915E-19"
-          izz="3.31951561015737E-07" />
+          value="0.025" />
       </inertial>
       <visual>
@@ -353,5 +297,5 @@
     </link>
     <joint
-      name="${end}_${side}_base_link_to_${end}_${side}_roller4"
+      name="${end}_${side}_wheel_to_${end}_${side}_roller4"
       type="continuous">
       <origin
@@ -359,5 +303,5 @@
         rpy="-0.59653 1.3924 -2.9492" />
       <parent
-        link="${end}_${side}_base_link" />
+        link="${end}_${side}_wheel" />
       <child
         link="${end}_${side}_roller4" />
@@ -372,12 +316,5 @@
           rpy="0 0 0" />
         <mass
-          value="0.00499543658848241" />
-        <inertia
-          ixx="8.99919949250993E-07"
-          ixy="3.14328632770151E-23"
-          ixz="7.25437397209005E-22"
-          iyy="8.99919949251052E-07"
-          iyz="-8.01796093915E-19"
-          izz="3.31951561019638E-07" />
+          value="0.025" />
       </inertial>
       <visual>
@@ -406,5 +343,5 @@
     </link>
     <joint
-      name="${end}_${side}_base_link_to_${end}_${side}_roller5"
+      name="${end}_${side}_wheel_to_${end}_${side}_roller5"
       type="continuous">
       <origin
@@ -412,5 +349,5 @@
         rpy="-0.73578 0.97593 -3.081" />
       <parent
-        link="${end}_${side}_base_link" />
+        link="${end}_${side}_wheel" />
       <child
         link="${end}_${side}_roller5" />
@@ -425,12 +362,5 @@
           rpy="0 0 0" />
         <mass
-          value="0.00499543658848228" />
-        <inertia
-          ixx="8.99919949249441E-07"
-          ixy="5.9557004103818E-23"
-          ixz="8.28834973778134E-22"
-          iyy="8.99919949249495E-07"
-          iyz="-8.017828590252E-19"
-          izz="3.31951561016508E-07" />
+          value="0.025" />
       </inertial>
       <visual>
@@ -459,5 +389,5 @@
     </link>
     <joint
-      name="${end}_${side}_base_link_to_${end}_${side}_roller6"
+      name="${end}_${side}_wheel_to_${end}_${side}_roller6"
       type="continuous">
       <origin
@@ -465,5 +395,5 @@
         rpy="-0.76481 0.55754 -3.1016" />
       <parent
-        link="${end}_${side}_base_link" />
+        link="${end}_${side}_wheel" />
       <child
         link="${end}_${side}_roller6" />
@@ -478,12 +408,5 @@
           rpy="0 0 0" />
         <mass
-          value="0.00499543658848228" />
-        <inertia
-          ixx="8.9991994924911E-07"
-          ixy="-3.30872245021211E-24"
-          ixz="7.51079996198149E-22"
-          iyy="8.99919949249103E-07"
-          iyz="-8.00353490926708E-19"
-          izz="3.31951561015786E-07" />
+          value="0.025" />
       </inertial>
       <visual>
@@ -512,5 +435,5 @@
     </link>
     <joint
-      name="${end}_${side}_base_link_to_${end}_${side}_roller7"
+      name="${end}_${side}_wheel_to_${end}_${side}_roller7"
       type="continuous">
       <origin
@@ -518,5 +441,5 @@
         rpy="-0.78123 0.13894 -3.1073" />
       <parent
-        link="${end}_${side}_base_link" />
+        link="${end}_${side}_wheel" />
       <child
         link="${end}_${side}_roller7" />
@@ -531,12 +454,5 @@
           rpy="0 0 0" />
         <mass
-          value="0.00499543658848253" />
-        <inertia
-          ixx="8.9991994925561E-07"
-          ixy="-4.13590306276514E-23"
-          ixz="7.46944093135384E-22"
-          iyy="8.99919949255578E-07"
-          iyz="-8.01624040347589E-19"
-          izz="3.31951561027997E-07" />
+          value="0.025" />
       </inertial>
       <visual>
@@ -565,5 +481,5 @@
     </link>
     <joint
-      name="${end}_${side}_base_link_to_${end}_${side}_roller8"
+      name="${end}_${side}_wheel_to_${end}_${side}_roller8"
       type="continuous">
       <origin
@@ -571,5 +487,5 @@
         rpy="-0.79573 -0.27969 -3.1063" />
       <parent
-        link="${end}_${side}_base_link" />
+        link="${end}_${side}_wheel" />
       <child
         link="${end}_${side}_roller8" />
@@ -584,12 +500,5 @@
           rpy="0 0 0" />
         <mass
-          value="0.00499543658848228" />
-        <inertia
-          ixx="8.99919949250354E-07"
-          ixy="1.81979734761666E-22"
-          ixz="8.08982639076861E-22"
-          iyy="8.99919949250367E-07"
-          iyz="-8.01835798584403E-19"
-          izz="3.31951561017902E-07" />
+          value="0.025" />
       </inertial>
       <visual>
@@ -618,5 +527,5 @@
     </link>
     <joint
-      name="${end}_${side}_base_link_to_${end}_${side}_roller9"
+      name="${end}_${side}_wheel_to_${end}_${side}_roller9"
       type="continuous">
       <origin
@@ -624,5 +533,5 @@
         rpy="-0.81448 -0.69826 -3.0973" />
       <parent
-        link="${end}_${side}_base_link" />
+        link="${end}_${side}_wheel" />
       <child
         link="${end}_${side}_roller9" />
@@ -637,12 +546,5 @@
           rpy="0 0 0" />
         <mass
-          value="0.00499543658848228" />
-        <inertia
-          ixx="8.99919949250464E-07"
-          ixy="-1.43929426584227E-22"
-          ixz="8.58613475830043E-22"
-          iyy="8.99919949250483E-07"
-          iyz="-8.01756389245598E-19"
-          izz="3.31951561018128E-07" />
+          value="0.025" />
       </inertial>
       <visual>
@@ -671,5 +573,5 @@
     </link>
     <joint
-      name="${end}_${side}_base_link_to_${end}_${side}_roller10"
+      name="${end}_${side}_wheel_to_${end}_${side}_roller10"
       type="continuous">
       <origin
@@ -677,5 +579,5 @@
         rpy="-0.85554 -1.1164 -3.0642" />
       <parent
-        link="${end}_${side}_base_link" />
+        link="${end}_${side}_wheel" />
       <child
         link="${end}_${side}_roller10" />
@@ -690,12 +592,5 @@
           rpy="0 0 0" />
         <mass
-          value="0.00499543658848228" />
-        <inertia
-          ixx="8.99919949249114E-07"
-          ixy="-6.61744490042422E-24"
-          ixz="8.13118542139626E-22"
-          iyy="8.99919949249044E-07"
-          iyz="-8.00419665375712E-19"
-          izz="3.31951561015731E-07" />
+          value="0.025" />
       </inertial>
       <visual>
@@ -724,5 +619,5 @@
     </link>
     <joint
-      name="${end}_${side}_base_link_to_${end}_${side}_roller11"
+      name="${end}_${side}_wheel_to_${end}_${side}_roller11"
       type="continuous">
       <origin
@@ -730,5 +625,5 @@
         rpy="-1.5658 -1.5225 -2.3612" />
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