Commit message: Added a lot of damping to wheel joints to minimize robot bumpiness

File: linorobot2_description/urdf/mech/mecanum_wheel_right.urdf.xacro (robot description, xacro)
@@ -2,5 +2,5 @@
 <robot xmlns:xacro="http://ros.org/wiki/xacro">
   <xacro:macro name="mecanum_wheel_right" params="side end radius width pos_x pos_y pos_z mass">
-    <link name="${end}_${side}_base_link">
+    <link name="${end}_${side}_wheel">
       <inertial>
         <origin
@@ -8,12 +8,5 @@
           rpy="0 0 0" />
         <mass
-          value="0.0396439871820506" />
-        <inertia
-          ixx="3.76805204137311E-05"
-          ixy="1.66580607308995E-20"
-          ixz="3.71031510257902E-18"
-          iyy="3.76805204137311E-05"
-          iyz="1.63812405352096E-18"
-          izz="7.1054120055567E-05" />
+          value="0.25" />
       </inertial>
       <visual>
@@ -41,8 +34,8 @@
       </collision>
     </link>
-    <joint name="base_link_to_${end}_${side}_base_link" type="continuous">
+    <joint name="base_link_to_${end}_${side}_wheel" type="continuous">
       <origin xyz="${pos_x} ${pos_y} 0"  rpy="0 0 0" />
       <parent link="base_link" />
-      <child link="${end}_${side}_base_link" />
+      <child link="${end}_${side}_wheel" />
       <axis xyz="0 1 0" />
     </joint>
@@ -54,12 +47,5 @@
           rpy="0 0 0" />
         <mass
-          value="0.0396439871820506" />
-        <inertia
-          ixx="7.1054120055567E-05"
-          ixy="1.62690471844664E-18"
-          ixz="-3.70636817664487E-18"
-          iyy="3.76805204137311E-05"
-          iyz="1.0973915143622E-20"
-          izz="3.76805204137311E-05" />
+          value="0.5" />
       </inertial>
       <visual>
@@ -88,5 +74,5 @@
     </link>
     <joint
-      name="${end}_${side}_base_link_to_drum"
+      name="${end}_${side}_wheel_to_drum"
       type="fixed">
       <origin
@@ -94,5 +80,5 @@
         rpy="1.5707963267949 0 -1.5707963267949" />
       <parent
-        link="${end}_${side}_base_link" />
+        link="${end}_${side}_wheel" />
       <child
         link="${end}_${side}_drum" />
@@ -103,16 +89,5 @@
       name="${end}_${side}_plate1">
       <inertial>
-        <origin
-          xyz="-0.00283756867072453 8.89413056967719E-16 2.68096171575045E-15"
-          rpy="0 0 0" />
-        <mass
-          value="0.0253986639693881" />
-        <inertia
-          ixx="8.39719993847471E-05"
-          ixy="1.90079838330856E-18"
-          ixz="4.7133202434868E-18"
-          iyy="4.21627753206921E-05"
-          iyz="-1.48230765769502E-20"
-          izz="4.21627753206921E-05" />
+        <mass value="0.5" />
       </inertial>
       <visual>
@@ -141,5 +116,5 @@
     </link>
     <joint
-      name="${end}_${side}_base_link_to_${end}_${side}_plate1"
+      name="${end}_${side}_wheel_to_${end}_${side}_plate1"
       type="fixed">
       <origin
@@ -147,5 +122,5 @@
         rpy="-1.60435101016735 0 1.5707963267949" />
       <parent
-        link="${end}_${side}_base_link" />
+        link="${end}_${side}_wheel" />
       <child
         link="${end}_${side}_plate1" />
@@ -156,16 +131,5 @@
       name="${end}_${side}_plate2">
       <inertial>
-        <origin
-          xyz="-0.00283756867072453 -9.8249688244021E-17 5.89771118826868E-17"
-          rpy="0 0 0" />
-        <mass
-          value="0.0253986639693881" />
-        <inertia
-          ixx="8.39719993847471E-05"
-          ixy="-9.13983660820293E-21"
-          ixz="5.31128745957199E-22"
-          iyy="4.2162775320692E-05"
-          iyz="1.59877468794249E-20"
-          izz="4.21627753206921E-05" />
+        <mass value="0.5" />
       </inertial>
       <visual>
@@ -194,5 +158,5 @@
     </link>
     <joint
-      name="${end}_${side}_base_link_to_${end}_${side}_plate2"
+      name="${end}_${side}_wheel_to_${end}_${side}_plate2"
       type="fixed">
       <origin
@@ -200,5 +164,5 @@
         rpy="1.60435101016734 0 -1.5707963267949" />
       <parent
-        link="${end}_${side}_base_link" />
+        link="${end}_${side}_wheel" />
       <child
         link="${end}_${side}_plate2" />
@@ -213,12 +177,5 @@
           rpy="0 0 0" />
         <mass
-          value="0.00499543658848254" />
-        <inertia
-          ixx="8.99919949255961E-07"
-          ixy="0"
-          ixz="7.14684049245816E-22"
-          iyy="8.999199492559E-07"
-          iyz="-8.01670362461892E-19"
-          izz="3.31951561028667E-07" />
+          value="0.025" />
       </inertial>
       <visual>
@@ -247,5 +204,5 @@
     </link>
     <joint
-      name="${end}_${side}_base_link_to_${end}_${side}_roller1"
+      name="${end}_${side}_wheel_to_${end}_${side}_roller1"
       type="continuous">
       <origin
@@ -253,5 +210,5 @@
         rpy="-2.36778917303694 -0.95454994461673 -1.76416393166909" />
       <parent
-        link="${end}_${side}_base_link" />
+        link="${end}_${side}_wheel" />
       <child
         link="${end}_${side}_roller1" />
@@ -266,12 +223,5 @@
           rpy="0 0 0" />
         <mass
-          value="0.00499543658848222" />
-        <inertia
-          ixx="8.99919949249302E-07"
-          ixy="-1.32348898008484E-22"
-          ixz="5.16160702233089E-22"
-          iyy="8.99919949249335E-07"
-          iyz="-8.02001234706914E-19"
-          izz="3.31951561015819E-07" />
+          value="0.025" />
       </inertial>
       <visual>
@@ -300,5 +250,5 @@
     </link>
     <joint
-      name="${end}_${side}_base_link_to_${end}_${side}_roller2"
+      name="${end}_${side}_wheel_to_${end}_${side}_roller2"
       type="continuous">
       <origin
@@ -306,5 +256,5 @@
         rpy="-1.77439072812908 -0.775855866169197 -2.22324127737972" />
       <parent
-        link="${end}_${side}_base_link" />
+        link="${end}_${side}_wheel" />
       <child
         link="${end}_${side}_roller2" />
@@ -319,12 +269,5 @@
           rpy="0 0 0" />
         <mass
-          value="0.00499543658848234" />
-        <inertia
-          ixx="8.99919949252429E-07"
-          ixy="-1.45583787809333E-22"
-          ixz="6.48509600241574E-22"
-          iyy="8.9991994925244E-07"
-          iyz="-8.05501863059238E-19"
-          izz="3.3195156102205E-07" />
+          value="0.025" />
       </inertial>
       <visual>
@@ -353,5 +296,5 @@
     </link>
     <joint
-      name="${end}_${side}_base_link_to_${end}_${side}_roller3"
+      name="${end}_${side}_wheel_to_${end}_${side}_roller3"
       type="continuous">
       <origin
@@ -359,5 +302,5 @@
         rpy="-1.40103696999546 -0.48194994387805 -2.44694050545059" />
       <parent
-        link="${end}_${side}_base_link" />
+        link="${end}_${side}_wheel" />
       <child
         link="${end}_${side}_roller3" />
@@ -372,12 +315,5 @@
           rpy="0 0 0" />
         <mass
-          value="0.00499543658848215" />
-        <inertia
-          ixx="8.99919949244641E-07"
-          ixy="0"
-          ixz="8.73502726855997E-22"
-          iyy="8.99919949244639E-07"
-          iyz="-8.01855650919104E-19"
-          izz="3.31951561007608E-07" />
+          value="0.025" />
       </inertial>
       <visual>
@@ -406,5 +342,5 @@
     </link>
     <joint
-      name="${end}_${side}_base_link_to_${end}_${side}_roller4"
+      name="${end}_${side}_wheel_to_${end}_${side}_roller4"
       type="continuous">
       <origin
@@ -412,5 +348,5 @@
         rpy="-1.13469826196558 -0.147073422491862 -2.53094960861872" />
       <parent
-        link="${end}_${side}_base_link" />
+        link="${end}_${side}_wheel" />
       <child
         link="${end}_${side}_roller4" />
@@ -425,12 +361,5 @@
           rpy="0 0 0" />
         <mass
-          value="0.00499543658848228" />
-        <inertia
-          ixx="8.99919949249555E-07"
-          ixy="-7.94093388050907E-23"
-          ixz="9.26442286059391E-22"
-          iyy="8.99919949249567E-07"
-          iyz="-8.01729919465996E-19"
-          izz="3.31951561016665E-07" />
+          value="0.025" />
       </inertial>
       <visual>
@@ -459,5 +388,5 @@
     </link>
     <joint
-      name="${end}_${side}_base_link_to_${end}_${side}_roller5"
+      name="${end}_${side}_wheel_to_${end}_${side}_roller5"
       type="continuous">
       <origin
@@ -465,5 +394,5 @@
         rpy="-0.894575475762315 0.197031441859666 -2.52483292758441" />
       <parent
-        link="${end}_${side}_base_link" />
+        link="${end}_${side}_wheel" />
       <child
         link="${end}_${side}_roller5" />
@@ -478,12 +407,5 @@
           rpy="0 0 0" />
         <mass
-          value="0.00499543658848248" />
-        <inertia
-          ixx="8.99919949253375E-07"
-          ixy="-1.05879118406788E-22"
-          ixz="8.73502726855997E-22"
-          iyy="8.99919949253382E-07"
-          iyz="-8.01961530037511E-19"
-          izz="3.31951561023958E-07" />
+          value="0.025" />
       </inertial>
       <visual>
@@ -512,5 +434,5 @@
     </link>
     <joint
-      name="${end}_${side}_base_link_to_${end}_${side}_roller6"
+      name="${end}_${side}_wheel_to_${end}_${side}_roller6"
       type="continuous">
       <origin
@@ -518,5 +440,5 @@
         rpy="-0.618670381864381 0.528470873009444 -2.42501713902796" />
       <parent
-        link="${end}_${side}_base_link" />
+        link="${end}_${side}_wheel" />
       <child
         link="${end}_${side}_roller6" />
@@ -531,12 +453,5 @@
           rpy="0 0 0" />
         <mass
-          value="0.00499543658848216" />
-        <inertia
-          ixx="8.99919949243988E-07"
-          ixy="-1.58818677610181E-22"
-          ixz="6.88214269644119E-22"
-          iyy="8.99919949243943E-07"
-          iyz="-8.01842416029303E-19"
-          izz="3.31951561006258E-07" />
+          value="0.025" />
       </inertial>
       <visual>
@@ -565,5 +480,5 @@
     </link>
     <joint
-      name="${end}_${side}_base_link_to_${end}_${side}_roller7"
+      name="${end}_${side}_wheel_to_${end}_${side}_roller7"
       type="continuous">
       <origin
@@ -571,5 +486,5 @@
         rpy="-0.22003525595071 0.81173834281584 -2.17291203984087" />
       <parent
-        link="${end}_${side}_base_link" />
+        link="${end}_${side}_wheel" />
       <child
         link="${end}_${side}_roller7" />
@@ -584,12 +499,5 @@
           rpy="0 0 0" />
         <mass
-          value="0.00499543658848215" />
-        <inertia
-          ixx="8.99919949245218E-07"
-          ixy="-2.64697796016969E-23"
-          ixz="7.94093388050907E-22"
-          iyy="8.99919949245208E-07"
-          iyz="-8.02067409155918E-19"
-          izz="3.31951561008361E-07" />
+          value="0.025" />
       </inertial>
       <visual>
@@ -618,5 +526,5 @@
     </link>
     <joint
-      name="${end}_${side}_base_link_to_${end}_${side}_roller8"
+      name="${end}_${side}_wheel_to_${end}_${side}_roller8"
       type="continuous">
       <origin
@@ -624,5 +532,5 @@
         rpy="0.408043134594723 0.963708851734786 -1.67797755478808" />
       <parent
-        link="${end}_${side}_base_link" />
+        link="${end}_${side}_wheel" />
       <child
         link="${end}_${side}_roller8" />
@@ -637,12 +545,5 @@
           rpy="0 0 0" />
         <mass
-          value="0.00499543658848229" />
-        <inertia
-          ixx="8.9991994924954E-07"
-          ixy="-2.64697796016969E-23"
-          ixz="7.6762360844921E-22"
-          iyy="8.99919949249544E-07"
-          iyz="-8.01743154355797E-19"
-          izz="3.31951561016627E-07" />
+          value="0.025" />
       </inertial>
       <visual>
@@ -671,5 +572,5 @@
     </link>
     <joint
-      name="${end}_${side}_base_link_to_${end}_${side}_roller9"
+      name="${end}_${side}_wheel_to_${end}_${side}_roller9"
       type="continuous">
       <origin
@@ -677,5 +578,5 @@
         rpy="1.1026415771303 0.886919106568413 -1.11464531078552" />
       <parent
-        link="${end}_${side}_base_link" />
+        link="${end}_${side}_wheel" />
       <child
         link="${end}_${side}_roller9" />
@@ -690,12 +591,5 @@
           rpy="0 0 0" />
         <mass
-          value="0.00499543658848216" />
-        <inertia
-          ixx="8.99919949244339E-07"
-          ixy="-1.05879118406788E-22"
-          ixz="8.33798057453452E-22"
-          iyy="8.99919949244339E-07"
-          iyz="-8.05177608259117E-19"
-          izz="3.31951561007005E-07" />
+          value="0.025" />
       </inertial>
       <visual>
@@ -724,5 +618,5 @@
     </link>
     <joint
-      name="${end}_${side}_base_link_to_${end}_${side}_roller10"
+      name="${end}_${side}_wheel_to_${end}_${side}_roller10"
       type="continuous">
       <origin
@@ -730,5 +624,5 @@
         rpy="1.57421323203544 0.637163580624169 -0.783361608443036" />
       <parent
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
File: linorobot2_description/urdf/mech/side_channel.urdf.xacro (robot description, xacro)
@@ -16,4 +16,7 @@
         </geometry>
       </collision>
+      <inertial>
+        <mass value="5"/>
+      </inertial>
     </link>
     <joint name="base_link_to_${side}_channel" type="fixed">
