Commit message: All 4 wheels loaded into Isaacsim and linorobot2 doing mecanum-style movements

File: linorobot2_description/urdf/mech/mecanum_wheel_right.urdf.xacro (robot description, xacro)
@@ -41,9 +41,9 @@
       </collision>
     </link>
-    <joint name="base_link_to_${end}_${side}_base_link" type="fixed">
+    <joint name="base_link_to_${end}_${side}_base_link" type="continuous">
       <origin xyz="${pos_x} ${pos_y} 0"  rpy="0 0 0" />
       <parent link="base_link" />
       <child link="${end}_${side}_base_link" />
-      <axis xyz="0 0 0" />
+      <axis xyz="0 1 0" />
     </joint>
     <link
