Commit message: All 4 wheels loaded into Isaacsim and linorobot2 doing mecanum-style movements

File: linorobot2_description/urdf/robots/mecanum.urdf (robot description, URDF)
Before this commit: robot linorobot2_2wd, 20 links, 19 joints
Links:
- added link front_right_base_link, mass 0.0396439871820506; collision mesh filename=package://linorobot2_description/mecanum_wheel_right/meshes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; visual mesh filename=package://linorobot2_description/mecanum_wheel_right/meshes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
- added link front_right_drum, mass 0.0396439871820506; collision mesh filename=package://linorobot2_description/mecanum_wheel_right/meshes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; visual mesh filename=package://linorobot2_description/mecanum_wheel_right/meshes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
- added link front_right_plate1, mass 0.0253986639693881; collision mesh filename=package://linorobot2_description/mecanum_wheel_right/meshes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; visual mesh filename=package://linorobot2_description/mecanum_wheel_right/meshes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
- added link front_right_plate2, mass 0.0253986639693881; collision mesh filename=package://linorobot2_description/mecanum_wheel_right/meshes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; visual mesh filename=package://linorobot2_description/mecanum_wheel_right/meshes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
- added link front_right_roller1, mass 0.00499543658848254; collision mesh filename=package://linorobot2_description/mecanum_wheel_right/meshes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; visual mesh filename=package://linorobot2_description/mecanum_wheel_right/meshes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
- added link front_right_roller10, mass 0.00499543658848216; collision mesh filename=package://linorobot2_description/mecanum_wheel_right/meshes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; visual mesh filename=package://linorobot2_description/mecanum_wheel_right/meshes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
- added link front_right_roller11, mass 0.00499543658848235; collision mesh filename=package://linorobot2_description/mecanum_wheel_right/meshes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; visual mesh filename=package://linorobot2_description/mecanum_wheel_right/meshes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
- added link front_right_roller12, mass 0.00499543658848216; collision mesh filename=package://linorobot2_description/mecanum_wheel_right/meshes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; visual mesh filename=package://linorobot2_description/mecanum_wheel_right/meshes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
- added link front_right_roller13, mass 0.00499543658848228; collision mesh filename=package://linorobot2_description/mecanum_wheel_right/meshes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; visual mesh filename=package://linorobot2_description/mecanum_wheel_right/meshes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
- added link front_right_roller14, mass 0.00499543658848209; collision mesh filename=package://linorobot2_description/mecanum_wheel_right/meshes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; visual mesh filename=package://linorobot2_description/mecanum_wheel_right/meshes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
- added link front_right_roller15, mass 0.00499543658848241; collision mesh filename=package://linorobot2_description/mecanum_wheel_right/meshes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; visual mesh filename=package://linorobot2_description/mecanum_wheel_right/meshes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
- added link front_right_roller2, mass 0.00499543658848222; collision mesh filename=package://linorobot2_description/mecanum_wheel_right/meshes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; visual mesh filename=package://linorobot2_description/mecanum_wheel_right/meshes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
- added link front_right_roller3, mass 0.00499543658848234; collision mesh filename=package://linorobot2_description/mecanum_wheel_right/meshes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; visual mesh filename=package://linorobot2_description/mecanum_wheel_right/meshes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
- added link front_right_roller4, mass 0.00499543658848215; collision mesh filename=package://linorobot2_description/mecanum_wheel_right/meshes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; visual mesh filename=package://linorobot2_description/mecanum_wheel_right/meshes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
- added link front_right_roller5, mass 0.00499543658848228; collision mesh filename=package://linorobot2_description/mecanum_wheel_right/meshes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; visual mesh filename=package://linorobot2_description/mecanum_wheel_right/meshes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
- added link front_right_roller6, mass 0.00499543658848248; collision mesh filename=package://linorobot2_description/mecanum_wheel_right/meshes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; visual mesh filename=package://linorobot2_description/mecanum_wheel_right/meshes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
- added link front_right_roller7, mass 0.00499543658848216; collision mesh filename=package://linorobot2_description/mecanum_wheel_right/meshes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; visual mesh filename=package://linorobot2_description/mecanum_wheel_right/meshes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
- added link front_right_roller8, mass 0.00499543658848215; collision mesh filename=package://linorobot2_description/mecanum_wheel_right/meshes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; visual mesh filename=package://linorobot2_description/mecanum_wheel_right/meshes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
- added link front_right_roller9, mass 0.00499543658848229; collision mesh filename=package://linorobot2_description/mecanum_wheel_right/meshes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; visual mesh filename=package://linorobot2_description/mecanum_wheel_right/meshes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
- added link rear_left_base_link, mass 0.0396439871820506; collision mesh filename=package://linorobot2_description/mecanum_wheel_right/meshes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; visual mesh filename=package://linorobot2_description/mecanum_wheel_right/meshes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
- added link rear_left_drum, mass 0.0396439871820506; collision mesh filename=package://linorobot2_description/mecanum_wheel_right/meshes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; visual mesh filename=package://linorobot2_description/mecanum_wheel_right/meshes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
- added link rear_left_plate1, mass 0.0253986639693881; collision mesh filename=package://linorobot2_description/mecanum_wheel_right/meshes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; visual mesh filename=package://linorobot2_description/mecanum_wheel_right/meshes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
- added link rear_left_plate2, mass 0.0253986639693881; collision mesh filename=package://linorobot2_description/mecanum_wheel_right/meshes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; visual mesh filename=package://linorobot2_description/mecanum_wheel_right/meshes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
- added link rear_left_roller1, mass 0.00499543658848254; collision mesh filename=package://linorobot2_description/mecanum_wheel_right/meshes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; visual mesh filename=package://linorobot2_description/mecanum_wheel_right/meshes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
- added link rear_left_roller10, mass 0.00499543658848216; collision mesh filename=package://linorobot2_description/mecanum_wheel_right/meshes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; visual mesh filename=package://linorobot2_description/mecanum_wheel_right/meshes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
- added link rear_left_roller11, mass 0.00499543658848235; collision mesh filename=package://linorobot2_description/mecanum_wheel_right/meshes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; visual mesh filename=package://linorobot2_description/mecanum_wheel_right/meshes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
- added link rear_left_roller12, mass 0.00499543658848216; collision mesh filename=package://linorobot2_description/mecanum_wheel_right/meshes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; visual mesh filename=package://linorobot2_description/mecanum_wheel_right/meshes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
- added link rear_left_roller13, mass 0.00499543658848228; collision mesh filename=package://linorobot2_description/mecanum_wheel_right/meshes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; visual mesh filename=package://linorobot2_description/mecanum_wheel_right/meshes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
- added link rear_left_roller14, mass 0.00499543658848209; collision mesh filename=package://linorobot2_description/mecanum_wheel_right/meshes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; visual mesh filename=package://linorobot2_description/mecanum_wheel_right/meshes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
- added link rear_left_roller15, mass 0.00499543658848241; collision mesh filename=package://linorobot2_description/mecanum_wheel_right/meshes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; visual mesh filename=package://linorobot2_description/mecanum_wheel_right/meshes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
- added link rear_left_roller2, mass 0.00499543658848222; collision mesh filename=package://linorobot2_description/mecanum_wheel_right/meshes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; visual mesh filename=package://linorobot2_description/mecanum_wheel_right/meshes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
- added link rear_left_roller3, mass 0.00499543658848234; collision mesh filename=package://linorobot2_description/mecanum_wheel_right/meshes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; visual mesh filename=package://linorobot2_description/mecanum_wheel_right/meshes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
- added link rear_left_roller4, mass 0.00499543658848215; collision mesh filename=package://linorobot2_description/mecanum_wheel_right/meshes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; visual mesh filename=package://linorobot2_description/mecanum_wheel_right/meshes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
- added link rear_left_roller5, mass 0.00499543658848228; collision mesh filename=package://linorobot2_description/mecanum_wheel_right/meshes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; visual mesh filename=package://linorobot2_description/mecanum_wheel_right/meshes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
- added link rear_left_roller6, mass 0.00499543658848248; collision mesh filename=package://linorobot2_description/mecanum_wheel_right/meshes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; visual mesh filename=package://linorobot2_description/mecanum_wheel_right/meshes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
- added link rear_left_roller7, mass 0.00499543658848216; collision mesh filename=package://linorobot2_description/mecanum_wheel_right/meshes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; visual mesh filename=package://linorobot2_description/mecanum_wheel_right/meshes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
- added link rear_left_roller8, mass 0.00499543658848215; collision mesh filename=package://linorobot2_description/mecanum_wheel_right/meshes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; visual mesh filename=package://linorobot2_description/mecanum_wheel_right/meshes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
- added link rear_left_roller9, mass 0.00499543658848229; collision mesh filename=package://linorobot2_description/mecanum_wheel_right/meshes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; visual mesh filename=package://linorobot2_description/mecanum_wheel_right/meshes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
- added link rear_right_base_link, mass 0.039620820516108; collision mesh filename=package://linorobot2_description/mecanum_wheel_left/meshes/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; visual mesh filename=package://linorobot2_description/mecanum_wheel_left/meshes/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
- added link rear_right_plate1, mass 0.0253986639693882; collision mesh filename=package://linorobot2_description/mecanum_wheel_left/meshes/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; visual mesh filename=package://linorobot2_description/mecanum_wheel_left/meshes/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
- added link rear_right_plate2, mass 0.0253986639693882; collision mesh filename=package://linorobot2_description/mecanum_wheel_left/meshes/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; visual mesh filename=package://linorobot2_description/mecanum_wheel_left/meshes/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
- added link rear_right_roller1, mass 0.00499543658848208; collision mesh filename=package://linorobot2_description/mecanum_wheel_left/meshes/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; visual mesh filename=package://linorobot2_description/mecanum_wheel_left/meshes/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
- added link rear_right_roller10, mass 0.00499543658848228; collision mesh filename=package://linorobot2_description/mecanum_wheel_left/meshes/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; visual mesh filename=package://linorobot2_description/mecanum_wheel_left/meshes/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
- added link rear_right_roller11, mass 0.00499543658848228; collision mesh filename=package://linorobot2_description/mecanum_wheel_left/meshes/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; visual mesh filename=package://linorobot2_description/mecanum_wheel_left/meshes/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
- added link rear_right_roller12, mass 0.00499543658848222; collision mesh filename=package://linorobot2_description/mecanum_wheel_left/meshes/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; visual mesh filename=package://linorobot2_description/mecanum_wheel_left/meshes/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
- added link rear_right_roller13, mass 0.0049954365884824; collision mesh filename=package://linorobot2_description/mecanum_wheel_left/meshes/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; visual mesh filename=package://linorobot2_description/mecanum_wheel_left/meshes/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
- added link rear_right_roller14, mass 0.00499543658848228; collision mesh filename=package://linorobot2_description/mecanum_wheel_left/meshes/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; visual mesh filename=package://linorobot2_description/mecanum_wheel_left/meshes/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
- added link rear_right_roller15, mass 0.00499543658848229; collision mesh filename=package://linorobot2_description/mecanum_wheel_left/meshes/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; visual mesh filename=package://linorobot2_description/mecanum_wheel_left/meshes/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
- added link rear_right_roller2, mass 0.00499543658848216; collision mesh filename=package://linorobot2_description/mecanum_wheel_left/meshes/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; visual mesh filename=package://linorobot2_description/mecanum_wheel_left/meshes/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
- added link rear_right_roller3, mass 0.00499543658848228; collision mesh filename=package://linorobot2_description/mecanum_wheel_left/meshes/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; visual mesh filename=package://linorobot2_description/mecanum_wheel_left/meshes/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
- added link rear_right_roller4, mass 0.00499543658848229; collision mesh filename=package://linorobot2_description/mecanum_wheel_left/meshes/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; visual mesh filename=package://linorobot2_description/mecanum_wheel_left/meshes/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
- added link rear_right_roller5, mass 0.00499543658848241; collision mesh filename=package://linorobot2_description/mecanum_wheel_left/meshes/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; visual mesh filename=package://linorobot2_description/mecanum_wheel_left/meshes/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
- added link rear_right_roller6, mass 0.00499543658848228; collision mesh filename=package://linorobot2_description/mecanum_wheel_left/meshes/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; visual mesh filename=package://linorobot2_description/mecanum_wheel_left/meshes/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
- added link rear_right_roller7, mass 0.00499543658848228; collision mesh filename=package://linorobot2_description/mecanum_wheel_left/meshes/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; visual mesh filename=package://linorobot2_description/mecanum_wheel_left/meshes/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
- added link rear_right_roller8, mass 0.00499543658848253; collision mesh filename=package://linorobot2_description/mecanum_wheel_left/meshes/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; visual mesh filename=package://linorobot2_description/mecanum_wheel_left/meshes/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
- added link rear_right_roller9, mass 0.00499543658848228; collision mesh filename=package://linorobot2_description/mecanum_wheel_left/meshes/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; visual mesh filename=package://linorobot2_description/mecanum_wheel_left/meshes/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
Joints:
- added joint base_link_to_front_right_base_link: type continuous, parent base_link, child front_right_base_link, origin xyz=0.12 -0.1355 0 rpy=0 0 0, axis 0 1 0
- added joint base_link_to_rear_left_base_link: type continuous, parent base_link, child rear_left_base_link, origin xyz=-0.12 0.1355 0 rpy=0 0 0, axis 0 1 0
- added joint base_link_to_rear_right_base_link: type continuous, parent base_link, child rear_right_base_link, origin xyz=-0.12 -0.1355 0 rpy=0 0 0, axis 0 1 0
- added joint front_right_base_link_to_drum: type fixed, parent front_right_base_link, child front_right_drum, origin xyz=0 0 0 rpy=1.5707963267949 0 -1.5707963267949, axis 0 0 0
- added joint front_right_base_link_to_front_right_plate1: type fixed, parent front_right_base_link, child front_right_plate1, origin xyz=0 0.0254 0 rpy=-1.60435101016735 0 1.5707963267949, axis 0 0 0
- added joint front_right_base_link_to_front_right_plate2: type fixed, parent front_right_base_link, child front_right_plate2, origin xyz=0 -0.0254 0 rpy=1.60435101016734 0 -1.5707963267949, axis 0 0 0
- added joint front_right_base_link_to_front_right_roller1: type continuous, parent front_right_base_link, child front_right_roller1, origin xyz=0.0513105165568448 -0.0151129693198936 0.0444755356274741 rpy=-2.36778917303694 -0.95454994461673 -1.76416393166909, axis 0 0 1
- added joint front_right_base_link_to_front_right_roller10: type continuous, parent front_right_base_link, child front_right_roller10, origin xyz=-0.0153690159550034 -0.0151129693199065 -0.0661410290761748 rpy=1.57421323203544 0.637163580624169 -0.783361608443036, axis 0 0 1
- added joint front_right_base_link_to_front_right_roller11: type continuous, parent front_right_base_link, child front_right_roller11, origin xyz=0.0128616854218928 -0.0151129693199038 -0.0666739786332639 rpy=1.88109068595424 0.317129294370825 -0.639722033593165, axis 0 0 1
- added joint front_right_base_link_to_front_right_roller12: type continuous, parent front_right_base_link, child front_right_roller12, origin xyz=0.0388684845445997 -0.0151129693199006 -0.0556783915705813 rpy=2.12643201705665 -0.025160050703084 -0.60332516970669, axis 0 0 1
- added joint front_right_base_link_to_front_right_roller13: type continuous, parent front_right_base_link, child front_right_roller13, origin xyz=0.0581545695804492 -0.0151129693198971 -0.0350555047830372 rpy=2.37615666037905 -0.365916365141497 -0.652805521545524, axis 0 0 1
- added joint front_right_base_link_to_front_right_roller14: type continuous, parent front_right_base_link, child front_right_roller14, origin xyz=0.0673852012181607 -0.0151129693198943 -0.00837120274924246 rpy=2.69941973817462 -0.67973266586857 -0.817294146739146, axis 0 0 1
- added joint front_right_base_link_to_front_right_roller15: type continuous, parent front_right_base_link, child front_right_roller15, origin xyz=0.0649643193899178 -0.0151129693198934 0.0197605562898849 rpy=-3.077965161563 -0.911914057233449 -1.18487158274901, axis 0 0 1
- added joint front_right_base_link_to_front_right_roller2: type continuous, parent front_right_base_link, child front_right_roller2, origin xyz=0.0287846592696844 -0.0151129693198959 0.0615002908075162 rpy=-1.77439072812908 -0.775855866169197 -2.22324127737972, axis 0 0 1
- added joint front_right_base_link_to_front_right_roller3: type continuous, parent front_right_base_link, child front_right_roller3, origin xyz=0.00128167289437567 -0.0151129693198984 0.0678910869943366 rpy=-1.40103696999546 -0.48194994387805 -2.44694050545059, axis 0 0 1
- added joint front_right_base_link_to_front_right_roller4: type continuous, parent front_right_base_link, child front_right_roller4, origin xyz=-0.0264429263680024 -0.0151129693199014 0.062542897468674 rpy=-1.13469826196558 -0.147073422491862 -2.53094960861872, axis 0 0 1
- added joint front_right_base_link_to_front_right_roller5: type continuous, parent front_right_base_link, child front_right_roller5, origin xyz=-0.0495953034349089 -0.0151129693199047 0.0463804727862918 rpy=-0.894575475762315 0.197031441859666 -2.52483292758441, axis 0 0 1
- added joint front_right_base_link_to_front_right_roller6: type continuous, parent front_right_base_link, child front_right_roller6, origin xyz=-0.0641722019787319 -0.0151129693199074 0.0221984430057918 rpy=-0.618670381864381 0.528470873009444 -2.42501713902796, axis 0 0 1
- added joint front_right_base_link_to_front_right_roller7: type continuous, parent front_right_base_link, child front_right_roller7, origin xyz=-0.0676531438142786 -0.0151129693199092 -0.0058218992369328 rpy=-0.22003525595071 0.81173834281584 -2.17291203984087, axis 0 0 1
- added joint front_right_base_link_to_front_right_roller8: type continuous, parent front_right_base_link, child front_right_roller8, origin xyz=-0.0594362424748194 -0.0151129693199101 -0.0328355822112983 rpy=0.408043134594723 0.963708851734786 -1.67797755478808, axis 0 0 1
- added joint front_right_base_link_to_front_right_roller9: type continuous, parent front_right_base_link, child front_right_roller9, origin xyz=-0.0409422748501527 -0.015112969319909 -0.0541716947194296 rpy=1.1026415771303 0.886919106568413 -1.11464531078552, axis 0 0 1
- added joint rear_left_base_link_to_drum: type fixed, parent rear_left_base_link, child rear_left_drum, origin xyz=0 0 0 rpy=1.5707963267949 0 -1.5707963267949, axis 0 0 0
- added joint rear_left_base_link_to_rear_left_plate1: type fixed, parent rear_left_base_link, child rear_left_plate1, origin xyz=0 0.0254 0 rpy=-1.60435101016735 0 1.5707963267949, axis 0 0 0
- added joint rear_left_base_link_to_rear_left_plate2: type fixed, parent rear_left_base_link, child rear_left_plate2, origin xyz=0 -0.0254 0 rpy=1.60435101016734 0 -1.5707963267949, axis 0 0 0
- added joint rear_left_base_link_to_rear_left_roller1: type continuous, parent rear_left_base_link, child rear_left_roller1, origin xyz=0.0513105165568448 -0.0151129693198936 0.0444755356274741 rpy=-2.36778917303694 -0.95454994461673 -1.76416393166909, axis 0 0 1
- added joint rear_left_base_link_to_rear_left_roller10: type continuous, parent rear_left_base_link, child rear_left_roller10, origin xyz=-0.0153690159550034 -0.0151129693199065 -0.0661410290761748 rpy=1.57421323203544 0.637163580624169 -0.783361608443036, axis 0 0 1
- added joint rear_left_base_link_to_rear_left_roller11: type continuous, parent rear_left_base_link, child rear_left_roller11, origin xyz=0.0128616854218928 -0.0151129693199038 -0.0666739786332639 rpy=1.88109068595424 0.317129294370825 -0.639722033593165, axis 0 0 1
- added joint rear_left_base_link_to_rear_left_roller12: type continuous, parent rear_left_base_link, child rear_left_roller12, origin xyz=0.0388684845445997 -0.0151129693199006 -0.0556783915705813 rpy=2.12643201705665 -0.025160050703084 -0.60332516970669, axis 0 0 1
- added joint rear_left_base_link_to_rear_left_roller13: type continuous, parent rear_left_base_link, child rear_left_roller13, origin xyz=0.0581545695804492 -0.0151129693198971 -0.0350555047830372 rpy=2.37615666037905 -0.365916365141497 -0.652805521545524, axis 0 0 1
- added joint rear_left_base_link_to_rear_left_roller14: type continuous, parent rear_left_base_link, child rear_left_roller14, origin xyz=0.0673852012181607 -0.0151129693198943 -0.00837120274924246 rpy=2.69941973817462 -0.67973266586857 -0.817294146739146, axis 0 0 1
- added joint rear_left_base_link_to_rear_left_roller15: type continuous, parent rear_left_base_link, child rear_left_roller15, origin xyz=0.0649643193899178 -0.0151129693198934 0.0197605562898849 rpy=-3.077965161563 -0.911914057233449 -1.18487158274901, axis 0 0 1
- added joint rear_left_base_link_to_rear_left_roller2: type continuous, parent rear_left_base_link, child rear_left_roller2, origin xyz=0.0287846592696844 -0.0151129693198959 0.0615002908075162 rpy=-1.77439072812908 -0.775855866169197 -2.22324127737972, axis 0 0 1
- added joint rear_left_base_link_to_rear_left_roller3: type continuous, parent rear_left_base_link, child rear_left_roller3, origin xyz=0.00128167289437567 -0.0151129693198984 0.0678910869943366 rpy=-1.40103696999546 -0.48194994387805 -2.44694050545059, axis 0 0 1
- added joint rear_left_base_link_to_rear_left_roller4: type continuous, parent rear_left_base_link, child rear_left_roller4, origin xyz=-0.0264429263680024 -0.0151129693199014 0.062542897468674 rpy=-1.13469826196558 -0.147073422491862 -2.53094960861872, axis 0 0 1
- added joint rear_left_base_link_to_rear_left_roller5: type continuous, parent rear_left_base_link, child rear_left_roller5, origin xyz=-0.0495953034349089 -0.0151129693199047 0.0463804727862918 rpy=-0.894575475762315 0.197031441859666 -2.52483292758441, axis 0 0 1
- added joint rear_left_base_link_to_rear_left_roller6: type continuous, parent rear_left_base_link, child rear_left_roller6, origin xyz=-0.0641722019787319 -0.0151129693199074 0.0221984430057918 rpy=-0.618670381864381 0.528470873009444 -2.42501713902796, axis 0 0 1
- added joint rear_left_base_link_to_rear_left_roller7: type continuous, parent rear_left_base_link, child rear_left_roller7, origin xyz=-0.0676531438142786 -0.0151129693199092 -0.0058218992369328 rpy=-0.22003525595071 0.81173834281584 -2.17291203984087, axis 0 0 1
- added joint rear_left_base_link_to_rear_left_roller8: type continuous, parent rear_left_base_link, child rear_left_roller8, origin xyz=-0.0594362424748194 -0.0151129693199101 -0.0328355822112983 rpy=0.408043134594723 0.963708851734786 -1.67797755478808, axis 0 0 1
- added joint rear_left_base_link_to_rear_left_roller9: type continuous, parent rear_left_base_link, child rear_left_roller9, origin xyz=-0.0409422748501527 -0.015112969319909 -0.0541716947194296 rpy=1.1026415771303 0.886919106568413 -1.11464531078552, axis 0 0 1
- added joint rear_right_base_link_to_rear_right_plate1: type fixed, parent rear_right_base_link, child rear_right_plate1, origin xyz=0 0.023114 0 rpy=-1.5708 0.03287 0, axis 0 0 0
- added joint rear_right_base_link_to_rear_right_plate2: type fixed, parent rear_right_base_link, child rear_right_plate2, origin xyz=0 -0.023114 0 rpy=-1.5707963267949 0.0335546833724646 -3.14159265358979, axis 0 0 0
- added joint rear_right_base_link_to_rear_right_roller1: type continuous, parent rear_right_base_link, child rear_right_roller1, origin xyz=-0.064997 -0.01515 0.019737 rpy=2.3375 0.48899 -0.038445, axis 0 0 1
- added joint rear_right_base_link_to_rear_right_roller10: type continuous, parent rear_right_base_link, child rear_right_roller10, origin xyz=0.040982 -0.01515 -0.054171 rpy=-0.85554 -1.1164 -3.0642, axis 0 0 1
- added joint rear_right_base_link_to_rear_right_roller11: type continuous, parent rear_right_base_link, child rear_right_roller11, origin xyz=0.015406 -0.01515 -0.066157 rpy=-1.5658 -1.5225 -2.3612, axis 0 0 1
- added joint rear_right_base_link_to_rear_right_roller12: type continuous, parent rear_right_base_link, child rear_right_roller12, origin xyz=-0.012835 -0.01515 -0.066704 rpy=2.4393 -1.1848 -0.090248, axis 0 0 1
- added joint rear_right_base_link_to_rear_right_roller13: type continuous, parent rear_right_base_link, child rear_right_roller13, origin xyz=-0.038856 -0.01515 -0.055716 rpy=2.3883 -0.76678 -0.047134, axis 0 0 1
- added joint rear_right_base_link_to_rear_right_roller14: type continuous, parent rear_right_base_link, child rear_right_roller14, origin xyz=-0.058159 -0.01515 -0.035095 rpy=2.3679 -0.34825 -0.036106, axis 0 0 1
- added joint rear_right_base_link_to_rear_right_roller15: type continuous, parent rear_right_base_link, child rear_right_roller15, origin xyz=-0.0674050504299177 -0.0151497403158722 -0.00840608812639412 rpy=2.35322166168045 0.070379538766794 -0.0340216727613588, axis 0 0 1
- added joint rear_right_base_link_to_rear_right_roller2: type continuous, parent rear_right_base_link, child rear_right_roller2, origin xyz=-0.05135 -0.01515 0.044467 rpy=2.3122 0.90744 -0.055132, axis 0 0 1
- added joint rear_right_base_link_to_rear_right_roller3: type continuous, parent rear_right_base_link, child rear_right_roller3, origin xyz=-0.028824 -0.01515 0.061508 rpy=2.22 1.3248 -0.13976, axis 0 0 1
- added joint rear_right_base_link_to_rear_right_roller4: type continuous, parent rear_right_base_link, child rear_right_roller4, origin xyz=-0.0013143 -0.01515 0.067914 rpy=-0.59653 1.3924 -2.9492, axis 0 0 1
- added joint rear_right_base_link_to_rear_right_roller5: type continuous, parent rear_right_base_link, child rear_right_roller5, origin xyz=0.026423 -0.01515 0.062578 rpy=-0.73578 0.97593 -3.081, axis 0 0 1
- added joint rear_right_base_link_to_rear_right_roller6: type continuous, parent rear_right_base_link, child rear_right_roller6, origin xyz=0.049591 -0.01515 0.04642 rpy=-0.76481 0.55754 -3.1016, axis 0 0 1
- added joint rear_right_base_link_to_rear_right_roller7: type continuous, parent rear_right_base_link, child rear_right_roller7, origin xyz=0.064184 -0.01515 0.022237 rpy=-0.78123 0.13894 -3.1073, axis 0 0 1
- added joint rear_right_base_link_to_rear_right_roller8: type continuous, parent rear_right_base_link, child rear_right_roller8, origin xyz=0.06768 -0.01515 -0.0057919 rpy=-0.79573 -0.27969 -3.1063, axis 0 0 1
- added joint rear_right_base_link_to_rear_right_roller9: type continuous, parent rear_right_base_link, child rear_right_roller9, origin xyz=0.059473 -0.01515 -0.032819 rpy=-0.81448 -0.69826 -3.0973, axis 0 0 1
