Commit message: All 4 wheels loaded into Isaacsim and linorobot2 doing mecanum-style movements

File: linorobot2_description/urdf/robots/mecanum.urdf.xacro (robot description, xacro)
@@ -27,5 +27,5 @@
     mass="${wheel_mass}"
   />
-  <!-- <xacro:mecanum_wheel_right
+  <xacro:mecanum_wheel_right
     side="right"
     end="front"
@@ -36,7 +36,7 @@
     pos_z="${wheel_pos_z}"
     mass="${wheel_mass}"
-  /> -->
+  />
   <!-- Back wheels mechanum style swapped (left mecanum wheel goes on right side of robot, and vice versa) -->
-  <!-- <xacro:mecanum_wheel_right
+  <xacro:mecanum_wheel_right
     side="left"
     end="rear"
@@ -57,4 +57,4 @@
     pos_z="${wheel_pos_z}"
     mass="${wheel_mass}"
-  /> -->
+  />
 </robot>
