Commit message: got 4 mecanum wheels fixed onto linorobot2

File: linorobot2_description/urdf/mech/mecanum_wheel_left.urdf.xacro (robot description, xacro)
@@ -1,6 +1,6 @@
 <?xml version="1.0"?>
 <robot xmlns:xacro="http://ros.org/wiki/xacro">
-  <xacro:macro name="mecanum_wheel" params="mecanum_style end radius width pos_x pos_y pos_z mass">
-    <link name="${end}_${mecanum_style}_base_link">
+  <xacro:macro name="mecanum_wheel_left" params="side end radius width pos_x pos_y pos_z mass">
+    <link name="${end}_${side}_base_link">
       <inertial>
         <origin
@@ -23,5 +23,5 @@
         <geometry>
           <mesh
-            filename="package://linorobot2_description/mecanum_wheel_${mecanum_style}/meshes/base_link.STL" />
+            filename="package://linorobot2_description/mecanum_wheel_left/meshes/base_link.STL" />
         </geometry>
         <material
@@ -37,16 +37,16 @@
         <geometry>
           <mesh
-            filename="package://linorobot2_description/mecanum_wheel_${mecanum_style}/meshes/base_link.STL" />
-        </geometry>
-      </collision>
-    </link>
-    <joint name="base_link_to_${end}_${mecanum_style}_base_link" type="fixed">
+            filename="package://linorobot2_description/mecanum_wheel_left/meshes/base_link.STL" />
+        </geometry>
+      </collision>
+    </link>
+    <joint name="base_link_to_${end}_${side}_base_link" type="fixed">
       <origin xyz="${pos_x} ${pos_y} 0"  rpy="0 0 0" />
       <parent link="base_link" />
-      <child link="${end}_${mecanum_style}_base_link" />
+      <child link="${end}_${side}_base_link" />
       <axis xyz="0 0 0" />
     </joint>
     <link
-      name="${end}_${mecanum_style}_plate1">
+      name="${end}_${side}_plate1">
       <inertial>
         <origin
@@ -69,5 +69,5 @@
         <geometry>
           <mesh
-            filename="package://linorobot2_description/mecanum_wheel_${mecanum_style}/meshes/plate1.STL" />
+            filename="package://linorobot2_description/mecanum_wheel_left/meshes/plate1.STL" />
         </geometry>
         <material
@@ -83,10 +83,10 @@
         <geometry>
           <mesh
-            filename="package://linorobot2_description/mecanum_wheel_${mecanum_style}/meshes/plate1.STL" />
-        </geometry>
-      </collision>
-    </link>
-    <joint
-      name="${end}_${mecanum_style}_base_link_to_${end}_${mecanum_style}_plate1"
+            filename="package://linorobot2_description/mecanum_wheel_left/meshes/plate1.STL" />
+        </geometry>
+      </collision>
+    </link>
+    <joint
+      name="${end}_${side}_base_link_to_${end}_${side}_plate1"
       type="fixed">
       <origin
@@ -94,12 +94,12 @@
         rpy="-1.5708 0.03287 0" />
       <parent
-        link="${end}_${mecanum_style}_base_link" />
-      <child
-        link="${end}_${mecanum_style}_plate1" />
+        link="${end}_${side}_base_link" />
+      <child
+        link="${end}_${side}_plate1" />
       <axis
         xyz="0 0 0" />
     </joint>
     <link
-      name="${end}_${mecanum_style}_plate2">
+      name="${end}_${side}_plate2">
       <inertial>
         <origin
@@ -122,5 +122,5 @@
         <geometry>
           <mesh
-            filename="package://linorobot2_description/mecanum_wheel_${mecanum_style}/meshes/plate2.STL" />
+            filename="package://linorobot2_description/mecanum_wheel_left/meshes/plate2.STL" />
         </geometry>
         <material
@@ -136,10 +136,10 @@
         <geometry>
           <mesh
-            filename="package://linorobot2_description/mecanum_wheel_${mecanum_style}/meshes/plate2.STL" />
-        </geometry>
-      </collision>
-    </link>
-    <joint
-      name="${end}_${mecanum_style}_base_link_to_${end}_${mecanum_style}_plate2"
+            filename="package://linorobot2_description/mecanum_wheel_left/meshes/plate2.STL" />
+        </geometry>
+      </collision>
+    </link>
+    <joint
+      name="${end}_${side}_base_link_to_${end}_${side}_plate2"
       type="fixed">
       <origin
@@ -147,12 +147,12 @@
         rpy="-1.5707963267949 0.0335546833724646 -3.14159265358979" />
       <parent
-        link="${end}_${mecanum_style}_base_link" />
-      <child
-        link="${end}_${mecanum_style}_plate2" />
+        link="${end}_${side}_base_link" />
+      <child
+        link="${end}_${side}_plate2" />
       <axis
         xyz="0 0 0" />
     </joint>
     <link
-      name="${end}_${mecanum_style}_roller1">
+      name="${end}_${side}_roller1">
       <inertial>
         <origin
@@ -175,24 +175,24 @@
         <geometry>
           <mesh
-            filename="package://linorobot2_description/mecanum_wheel_${mecanum_style}/meshes/roller1.STL" />
-        </geometry>
-        <material
-          name="">
-          <color
-            rgba="0.752941176470588 0.752941176470588 0.752941176470588 1" />
-        </material>
-      </visual>
-      <collision>
-        <origin
-          xyz="0 0 0"
-          rpy="0 0 0" />
-        <geometry>
-          <mesh
-            filename="package://linorobot2_description/mecanum_wheel_${mecanum_style}/meshes/roller1.STL" />
-        </geometry>
-      </collision>
-    </link>
-    <joint
-      name="${end}_${mecanum_style}_base_link_to_${end}_${mecanum_style}_roller1"
+            filename="package://linorobot2_description/mecanum_wheel_left/meshes/roller1.STL" />
+        </geometry>
+        <material
+          name="">
+          <color
+            rgba="0.752941176470588 0.752941176470588 0.752941176470588 1" />
+        </material>
+      </visual>
+      <collision>
+        <origin
+          xyz="0 0 0"
+          rpy="0 0 0" />
+        <geometry>
+          <mesh
+            filename="package://linorobot2_description/mecanum_wheel_left/meshes/roller1.STL" />
+        </geometry>
+      </collision>
+    </link>
+    <joint
+      name="${end}_${side}_base_link_to_${end}_${side}_roller1"
       type="continuous">
       <origin
@@ -200,12 +200,12 @@
         rpy="2.3375 0.48899 -0.038445" />
       <parent
-        link="${end}_${mecanum_style}_base_link" />
-      <child
-        link="${end}_${mecanum_style}_roller1" />
-      <axis
-        xyz="0 0 1" />
-    </joint>
-    <link
-      name="${end}_${mecanum_style}_roller2">
+        link="${end}_${side}_base_link" />
+      <child
+        link="${end}_${side}_roller1" />
+      <axis
+        xyz="0 0 1" />
+    </joint>
+    <link
+      name="${end}_${side}_roller2">
       <inertial>
         <origin
@@ -228,24 +228,24 @@
         <geometry>
           <mesh
-            filename="package://linorobot2_description/mecanum_wheel_${mecanum_style}/meshes/roller2.STL" />
-        </geometry>
-        <material
-          name="">
-          <color
-            rgba="0.752941176470588 0.752941176470588 0.752941176470588 1" />
-        </material>
-      </visual>
-      <collision>
-        <origin
-          xyz="0 0 0"
-          rpy="0 0 0" />
-        <geometry>
-          <mesh
-            filename="package://linorobot2_description/mecanum_wheel_${mecanum_style}/meshes/roller2.STL" />
-        </geometry>
-      </collision>
-    </link>
-    <joint
-      name="${end}_${mecanum_style}_base_link_to_${end}_${mecanum_style}_roller2"
+            filename="package://linorobot2_description/mecanum_wheel_left/meshes/roller2.STL" />
+        </geometry>
+        <material
+          name="">
+          <color
+            rgba="0.752941176470588 0.752941176470588 0.752941176470588 1" />
+        </material>
+      </visual>
+      <collision>
+        <origin
+          xyz="0 0 0"
+          rpy="0 0 0" />
+        <geometry>
+          <mesh
+            filename="package://linorobot2_description/mecanum_wheel_left/meshes/roller2.STL" />
+        </geometry>
+      </collision>
+    </link>
+    <joint
+      name="${end}_${side}_base_link_to_${end}_${side}_roller2"
       type="continuous">
       <origin
@@ -253,12 +253,12 @@
         rpy="2.3122 0.90744 -0.055132" />
       <parent
-        link="${end}_${mecanum_style}_base_link" />
-      <child
-        link="${end}_${mecanum_style}_roller2" />
-      <axis
-        xyz="0 0 1" />
-    </joint>
-    <link
-      name="${end}_${mecanum_style}_roller3">
+        link="${end}_${side}_base_link" />
+      <child
+        link="${end}_${side}_roller2" />
+      <axis
+        xyz="0 0 1" />
+    </joint>
+    <link
+      name="${end}_${side}_roller3">
       <inertial>
         <origin
@@ -281,24 +281,24 @@
         <geometry>
           <mesh
-            filename="package://linorobot2_description/mecanum_wheel_${mecanum_style}/meshes/roller3.STL" />
-        </geometry>
-        <material
-          name="">
-          <color
-            rgba="0.752941176470588 0.752941176470588 0.752941176470588 1" />
-        </material>
-      </visual>
-      <collision>
-        <origin
-          xyz="0 0 0"
-          rpy="0 0 0" />
-        <geometry>
-          <mesh
-            filename="package://linorobot2_description/mecanum_wheel_${mecanum_style}/meshes/roller3.STL" />
-        </geometry>
-      </collision>
-    </link>
-    <joint
-      name="${end}_${mecanum_style}_base_link_to_${end}_${mecanum_style}_roller3"
+            filename="package://linorobot2_description/mecanum_wheel_left/meshes/roller3.STL" />
+        </geometry>
+        <material
+          name="">
+          <color
+            rgba="0.752941176470588 0.752941176470588 0.752941176470588 1" />
+        </material>
+      </visual>
+      <collision>
+        <origin
+          xyz="0 0 0"
+          rpy="0 0 0" />
+        <geometry>
+          <mesh
+            filename="package://linorobot2_description/mecanum_wheel_left/meshes/roller3.STL" />
+        </geometry>
+      </collision>
+    </link>
+    <joint
+      name="${end}_${side}_base_link_to_${end}_${side}_roller3"
       type="continuous">
       <origin
@@ -306,12 +306,12 @@
         rpy="2.22 1.3248 -0.13976" />
       <parent
-        link="${end}_${mecanum_style}_base_link" />
-      <child
-        link="${end}_${mecanum_style}_roller3" />
-      <axis
-        xyz="0 0 1" />
-    </joint>
-    <link
-      name="${end}_${mecanum_style}_roller4">
+        link="${end}_${side}_base_link" />
+      <child
+        link="${end}_${side}_roller3" />
+      <axis
+        xyz="0 0 1" />
+    </joint>
+    <link
+      name="${end}_${side}_roller4">
       <inertial>
         <origin
@@ -334,24 +334,24 @@
         <geometry>
           <mesh
-            filename="package://linorobot2_description/mecanum_wheel_${mecanum_style}/meshes/roller4.STL" />
-        </geometry>
-        <material
-          name="">
-          <color
-            rgba="0.752941176470588 0.752941176470588 0.752941176470588 1" />
-        </material>
-      </visual>
-      <collision>
-        <origin
-          xyz="0 0 0"
-          rpy="0 0 0" />
-        <geometry>
-          <mesh
-            filename="package://linorobot2_description/mecanum_wheel_${mecanum_style}/meshes/roller4.STL" />
-        </geometry>
-      </collision>
-    </link>
-    <joint
-      name="${end}_${mecanum_style}_base_link_to_${end}_${mecanum_style}_roller4"
+            filename="package://linorobot2_description/mecanum_wheel_left/meshes/roller4.STL" />
+        </geometry>
+        <material
+          name="">
+          <color
+            rgba="0.752941176470588 0.752941176470588 0.752941176470588 1" />
+        </material>
+      </visual>
+      <collision>
+        <origin
+          xyz="0 0 0"
+          rpy="0 0 0" />
+        <geometry>
+          <mesh
+            filename="package://linorobot2_description/mecanum_wheel_left/meshes/roller4.STL" />
+        </geometry>
+      </collision>
+    </link>
+    <joint
+      name="${end}_${side}_base_link_to_${end}_${side}_roller4"
       type="continuous">
       <origin
@@ -359,12 +359,12 @@
         rpy="-0.59653 1.3924 -2.9492" />
       <parent
-        link="${end}_${mecanum_style}_base_link" />
-      <child
-        link="${end}_${mecanum_style}_roller4" />
-      <axis
-        xyz="0 0 1" />
-    </joint>
-    <link
-      name="${end}_${mecanum_style}_roller5">
+        link="${end}_${side}_base_link" />
+      <child
+        link="${end}_${side}_roller4" />
+      <axis
+        xyz="0 0 1" />
+    </joint>
+    <link
+      name="${end}_${side}_roller5">
       <inertial>
         <origin
@@ -387,24 +387,24 @@
         <geometry>
           <mesh
-            filename="package://linorobot2_description/mecanum_wheel_${mecanum_style}/meshes/roller5.STL" />
-        </geometry>
-        <material
-          name="">
-          <color
-            rgba="0.752941176470588 0.752941176470588 0.752941176470588 1" />
-        </material>
-      </visual>
-      <collision>
-        <origin
-          xyz="0 0 0"
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
File: linorobot2_description/urdf/robots/mecanum.urdf.xacro (robot description, xacro)
@@ -3,5 +3,6 @@
   <xacro:include filename="$(find linorobot2_description)/urdf/mecanum_properties.urdf.xacro" />
   <xacro:include filename="$(find linorobot2_description)/urdf/mech/base.urdf.xacro" />
-  <xacro:include filename="$(find linorobot2_description)/urdf/mech/mecanum_wheel.urdf.xacro" />
+  <xacro:include filename="$(find linorobot2_description)/urdf/mech/mecanum_wheel_left.urdf.xacro" />
+  <xacro:include filename="$(find linorobot2_description)/urdf/mech/mecanum_wheel_right.urdf.xacro" />
   <xacro:include filename="$(find linorobot2_description)/urdf/sensors/imu.urdf.xacro" />
   <xacro:include filename="$(find linorobot2_description)/urdf/sensors/generic_laser.urdf.xacro" />
@@ -16,6 +17,6 @@
     wheel_pos_z="${wheel_pos_z}"
 />
-  <xacro:mecanum_wheel
-    mecanum_style="left"
+  <xacro:mecanum_wheel_left
+    side="left"
     end="front"
     radius="${wheel_radius}"
@@ -26,6 +27,7 @@
     mass="${wheel_mass}"
   />
-  <!-- <xacro:mecanum_wheel
-    mecanum_style="front_right"
+  <xacro:mecanum_wheel_right
+    side="right"
+    end="front"
     radius="${wheel_radius}"
     width="${wheel_width}"
@@ -34,7 +36,8 @@
     pos_z="${wheel_pos_z}"
     mass="${wheel_mass}"
-  /> -->
-  <!-- <xacro:mecanum_wheel
-    mecanum_style="left"
+  />
+  <!-- Back wheels mechanum style swapped (left mecanum wheel goes on right side of robot, and vice versa) -->
+  <xacro:mecanum_wheel_right
+    side="left"
     end="rear"
     radius="${wheel_radius}"
@@ -44,8 +47,7 @@
     pos_z="${wheel_pos_z}"
     mass="${wheel_mass}"
-  /> -->
-  <!-- Left style mecanum wheel is on back RIGHT of robot -->
-  <xacro:mecanum_wheel
-    mecanum_style="left"
+  />
+  <xacro:mecanum_wheel_left
+    side="right"
     end="rear"
     radius="${wheel_radius}"

Commit message: got one mecanum wheel spinning in isaacsim

File: linorobot2_description/urdf/mech/mecanum_wheel_left.urdf.xacro (robot description, xacro)
@@ -41,9 +41,9 @@
       </collision>
     </link>
-    <joint name="base_link_to_${end}_${side}_base_link" type="fixed">
+    <joint name="base_link_to_${end}_${side}_base_link" type="continuous">
       <origin xyz="${pos_x} ${pos_y} 0"  rpy="0 0 0" />
       <parent link="base_link" />
       <child link="${end}_${side}_base_link" />
-      <axis xyz="0 0 0" />
+      <axis xyz="0 1 0" />
     </joint>
     <link

File: linorobot2_description/urdf/robots/mecanum.urdf.xacro (robot description, xacro)
@@ -27,5 +27,5 @@
     mass="${wheel_mass}"
   />
-  <xacro:mecanum_wheel_right
+  <!-- <xacro:mecanum_wheel_right
     side="right"
     end="front"
@@ -36,7 +36,7 @@
     pos_z="${wheel_pos_z}"
     mass="${wheel_mass}"
-  />
+  /> -->
   <!-- Back wheels mechanum style swapped (left mecanum wheel goes on right side of robot, and vice versa) -->
-  <xacro:mecanum_wheel_right
+  <!-- <xacro:mecanum_wheel_right
     side="left"
     end="rear"
@@ -57,12 +57,4 @@
     pos_z="${wheel_pos_z}"
     mass="${wheel_mass}"
-  />
-  <xacro:imu/>
-  <xacro:generic_laser>
-    <xacro:insert_block name="laser_pose" />
-  </xacro:generic_laser>
-  <xacro:depth_sensor>
-    <xacro:insert_block name="depth_sensor_pose" />
-  </xacro:depth_sensor>
-  <xacro:omni_drive_controller/>
+  /> -->
 </robot>

Commit message: Added damping and friction to roller joints, robot moves more smoothly now

File: linorobot2_description/urdf/mech/mecanum_wheel_left.urdf.xacro (robot description, xacro)
@@ -39,4 +39,5 @@
       <child link="${end}_${side}_wheel" />
       <axis xyz="0 1 0" />
+      <dynamics damping="0.1" friction="0.01"/>
     </joint>
     <link
@@ -170,4 +171,5 @@
       <axis
         xyz="0 0 1" />
+      <dynamics damping="0.1" friction="0.01"/>
     </joint>
     <link
@@ -216,4 +218,5 @@
       <axis
         xyz="0 0 1" />
+      <dynamics damping="0.1" friction="0.01"/>
     </joint>
     <link
@@ -262,4 +265,5 @@
       <axis
         xyz="0 0 1" />
+      <dynamics damping="0.1" friction="0.01"/>
     </joint>
     <link
@@ -308,4 +312,5 @@
       <axis
         xyz="0 0 1" />
+      <dynamics damping="0.1" friction="0.01"/>
     </joint>
     <link
@@ -354,4 +359,5 @@
       <axis
         xyz="0 0 1" />
+      <dynamics damping="0.1" friction="0.01"/>
     </joint>
     <link
@@ -400,4 +406,5 @@
       <axis
         xyz="0 0 1" />
+      <dynamics damping="0.1" friction="0.01"/>
     </joint>
     <link
@@ -446,4 +453,5 @@
       <axis
         xyz="0 0 1" />
+      <dynamics damping="0.1" friction="0.01"/>
     </joint>
     <link
@@ -492,4 +500,5 @@
       <axis
         xyz="0 0 1" />
+      <dynamics damping="0.1" friction="0.01"/>
     </joint>
     <link
@@ -538,4 +547,5 @@
       <axis
         xyz="0 0 1" />
+      <dynamics damping="0.1" friction="0.01"/>
     </joint>
     <link
@@ -584,4 +594,5 @@
       <axis
         xyz="0 0 1" />
+      <dynamics damping="0.1" friction="0.01"/>
     </joint>
     <link
@@ -630,4 +641,5 @@
       <axis
         xyz="0 0 1" />
+      <dynamics damping="0.1" friction="0.01"/>
     </joint>
     <link
@@ -676,4 +688,5 @@
       <axis
         xyz="0 0 1" />
+      <dynamics damping="0.1" friction="0.01"/>
     </joint>
     <link
@@ -722,4 +735,5 @@
       <axis
         xyz="0 0 1" />
+      <dynamics damping="0.1" friction="0.01"/>
     </joint>
     <link
@@ -768,4 +782,5 @@
       <axis
         xyz="0 0 1" />
+      <dynamics damping="0.1" friction="0.01"/>
     </joint>
     <link
@@ -814,4 +829,5 @@
       <axis
         xyz="0 0 1" />
+      <dynamics damping="0.1" friction="0.01"/>
     </joint>
   </xacro:macro>

File: linorobot2_description/urdf/mech/mecanum_wheel_right.urdf.xacro (robot description, xacro)
@@ -215,4 +215,5 @@
       <axis
         xyz="0 0 1" />
+      <dynamics damping="0.1" friction="0.01"/>
     </joint>
     <link
@@ -261,4 +262,5 @@
       <axis
         xyz="0 0 1" />
+      <dynamics damping="0.1" friction="0.01"/>
     </joint>
     <link
@@ -307,4 +309,5 @@
       <axis
         xyz="0 0 1" />
+      <dynamics damping="0.1" friction="0.01"/>
     </joint>
     <link
@@ -353,4 +356,5 @@
       <axis
         xyz="0 0 1" />
+      <dynamics damping="0.1" friction="0.01"/>
     </joint>
     <link
@@ -399,4 +403,5 @@
       <axis
         xyz="0 0 1" />
+      <dynamics damping="0.1" friction="0.01"/>
     </joint>
     <link
@@ -445,4 +450,5 @@
       <axis
         xyz="0 0 1" />
+      <dynamics damping="0.1" friction="0.01"/>
     </joint>
     <link
@@ -491,4 +497,5 @@
       <axis
         xyz="0 0 1" />
+      <dynamics damping="0.1" friction="0.01"/>
     </joint>
     <link
@@ -537,4 +544,5 @@
       <axis
         xyz="0 0 1" />
+      <dynamics damping="0.1" friction="0.01"/>
     </joint>
     <link
@@ -583,4 +591,5 @@
       <axis
         xyz="0 0 1" />
+      <dynamics damping="0.1" friction="0.01"/>
     </joint>
     <link
@@ -629,4 +638,5 @@
       <axis
         xyz="0 0 1" />
+      <dynamics damping="0.1" friction="0.01"/>
     </joint>
     <link
@@ -675,4 +685,5 @@
       <axis
         xyz="0 0 1" />
+      <dynamics damping="0.1" friction="0.01"/>
     </joint>
     <link
@@ -721,4 +732,5 @@
       <axis
         xyz="0 0 1" />
+      <dynamics damping="0.1" friction="0.01"/>
     </joint>
     <link
@@ -767,4 +779,5 @@
       <axis
         xyz="0 0 1" />
+      <dynamics damping="0.1" friction="0.01"/>
     </joint>
     <link
@@ -813,4 +826,5 @@
       <axis
         xyz="0 0 1" />
+      <dynamics damping="0.1" friction="0.01"/>
     </joint>
     <link
@@ -859,4 +873,5 @@
       <axis
         xyz="0 0 1" />
+      <dynamics damping="0.1" friction="0.01"/>
     </joint>
   </xacro:macro>
