Commit message: Added front/back and left/right outer channels to drone URDF

File: linorobot2_description/urdf/mecanum_properties.urdf.xacro (robot description, xacro)
@@ -1,14 +1,14 @@
 <?xml version="1.0"?>
 <robot xmlns:xacro="http://ros.org/wiki/xacro">
-  <xacro:property name="base_length" value="0.445" />
-  <xacro:property name="base_width" value="0.200" />
-  <xacro:property name="base_height" value="0.129" />
-  <xacro:property name="base_mass" value="10" />
+  <xacro:property name="base_length" value="0.82067" />
+  <xacro:property name="base_width" value="0.3175" />
+  <xacro:property name="base_height" value="0.07772" />
+  <xacro:property name="base_mass" value="30" />
   <xacro:property name="wheel_radius" value="0.07162" />
   <xacro:property name="wheel_width" value="0.05" />
-  <xacro:property name="wheel_pos_x" value="0.120" />
-  <xacro:property name="wheel_pos_y" value="0.1355" />
-  <xacro:property name="wheel_pos_z" value="-0.04788" />
-  <xacro:property name="wheel_mass" value=".6" />
+  <xacro:property name="wheel_pos_x" value="0.25857" />
+  <xacro:property name="wheel_pos_y" value="0.19355" />
+  <xacro:property name="wheel_pos_z" value="0.0019" />
+  <xacro:property name="wheel_mass" value="2.0" />
   <xacro:property name="wheel_torque" value="20" />
   <xacro:property name="laser_pose">

File: linorobot2_description/urdf/mech/base.urdf.xacro (robot description, xacro)
@@ -10,6 +10,6 @@
           <!-- <mesh filename="" scale="0.001 0.001 0.001"/> -->
         </geometry>
-        <material name="yellow">
-          <color rgba="0.8784 0.6627 0.6627 1.0"/>
+        <material name="gray_base">
+          <color rgba="0.8 0.8 0.83 1.0"/>
         </material>
       </visual>

File: linorobot2_description/urdf/robots/mecanum.urdf (robot description, URDF)
Before this commit: robot linorobot2_2wd, 76 links, 75 joints
Links:
- added link back_channel; collision box size=0.05398 0.4953 0.08458; visual box size=0.05398 0.4953 0.08458
- added link front_channel; collision box size=0.05398 0.4953 0.08458; visual box size=0.05398 0.4953 0.08458
- added link left_channel; collision box size=0.82067 0.02224 0.07772; visual box size=0.82067 0.02224 0.07772
- added link right_channel; collision box size=0.82067 0.02224 0.07772; visual box size=0.82067 0.02224 0.07772
- link base_link: mass 10 -> 30; geometry collision box size=0.82067 0.3175 0.07772; visual box size=0.82067 0.3175 0.07772
Joints:
- added joint base_link_to_back_channel: type fixed, parent base_link, child back_channel, origin xyz=-0.383345 0 0 rpy=0 0 0
- added joint base_link_to_front_channel: type fixed, parent base_link, child front_channel, origin xyz=0.383345 0 0 rpy=0 0 0
- added joint base_link_to_left_channel: type fixed, parent base_link, child left_channel, origin xyz=0 0.23653 0 rpy=0 0 0
- added joint base_link_to_right_channel: type fixed, parent base_link, child right_channel, origin xyz=0 -0.23653 0 rpy=0 0 0
- joint base_link_to_front_left_base_link: origin xyz=0.12 0.1355 0 rpy=0 0 0 -> xyz=0.25857 0.19355 0 rpy=0 0 0
- joint base_link_to_front_right_base_link: origin xyz=0.12 -0.1355 0 rpy=0 0 0 -> xyz=0.25857 -0.19355 0 rpy=0 0 0
- joint base_link_to_rear_left_base_link: origin xyz=-0.12 0.1355 0 rpy=0 0 0 -> xyz=-0.25857 0.19355 0 rpy=0 0 0
- joint base_link_to_rear_right_base_link: origin xyz=-0.12 -0.1355 0 rpy=0 0 0 -> xyz=-0.25857 -0.19355 0 rpy=0 0 0
- joint base_to_footprint: origin xyz=0 0 0.1195 rpy=0 0 0 -> xyz=0 0 0.06972 rpy=0 0 0

File: linorobot2_description/urdf/robots/mecanum.urdf.xacro (robot description, xacro)
@@ -9,4 +9,6 @@
   <xacro:include filename="$(find linorobot2_description)/urdf/sensors/depth_sensor.urdf.xacro" />
   <xacro:include filename="$(find linorobot2_description)/urdf/controllers/omni_drive.urdf.xacro" />
+  <xacro:include filename="$(find linorobot2_description)/urdf/mech/end_channel.urdf.xacro" />
+  <xacro:include filename="$(find linorobot2_description)/urdf/mech/side_channel.urdf.xacro" />
   <xacro:base
     length="${base_length}"
@@ -16,5 +18,21 @@
     wheel_radius="${wheel_radius}"
     wheel_pos_z="${wheel_pos_z}"
-/>
+  />
+  <xacro:end_channel
+    end="front"
+    pos_x="0.383345"
+  />
+  <xacro:end_channel
+    end="back"
+    pos_x="-0.383345"
+  />
+  <xacro:side_channel
+    side="left"
+    pos_y="0.23653"
+  />
+  <xacro:side_channel
+    side="right"
+    pos_y="-0.23653"
+  />
   <xacro:mecanum_wheel_left
     side="left"
