Commit message: Added frames for simulated realsenses to URDF, but IsaacSim still needs them to be manually set in base link to realsense fixed joints, it doesnt parse the URDF properly

File: linorobot2_description/urdf/robots/mecanum.urdf (robot description, URDF)
Before this commit: robot linorobot2_mecanum, 80 links, 79 joints
Links:
- added link front_rs_depth_optical_frame, mass 0.025
- added link left_rs_depth_optical_frame, mass 0.025
- added link rear_rs_depth_optical_frame, mass 0.025
- added link right_rs_depth_optical_frame, mass 0.025
Joints:
- added joint base_link_to_front_rs: type fixed, parent base_link, child front_rs_depth_optical_frame, origin xyz=0.410335 0 0.0892 rpy=-1.57 1.57 0
- added joint base_link_to_left_rs: type fixed, parent base_link, child left_rs_depth_optical_frame, origin xyz=0 0.247 0.089 rpy=-1.57 0 0
- added joint base_link_to_rear_rs: type fixed, parent base_link, child rear_rs_depth_optical_frame, origin xyz=-0.41 0 0.089 rpy=-1.57 -1.57 0
- added joint base_link_to_right_rs: type fixed, parent base_link, child right_rs_depth_optical_frame, origin xyz=0 -0.247 0.089 rpy=1.57 0 3.14

File: linorobot2_description/urdf/robots/mecanum.urdf.xacro (robot description, xacro)
@@ -76,3 +76,26 @@
     mass="${wheel_mass}"
   />
+  <link name="front_rs_depth_optical_frame">
+    <inertial>
+      <mass value="0.025" />
+    </inertial>
+    <visual>
+      <origin
+        xyz="0 0 0"
+        rpy="0 0 0" />
+    </visual>
+    <collision>
+      <origin
+        xyz="0 0 0"
+        rpy="0 0 0" />
+    </collision>
+  </link>
+  <joint
+    name="base_link_to_front_rs" type="fixed">
+    <origin
+      xyz="0 0 0"
+      rpy="0 0 0" />
+    <parent link="base_link" />
+    <child link="front_rs_depth_optical_frame" />
+  </joint>
 </robot>
