Commit message: Constrained pointcloud angles when turning to scans, since they will need to be merged into one scan without overlapping sections. Rear realsense had to be split into two, due to angle crossing at pi/-pi

File: linorobot2_description/urdf/robots/mecanum.urdf.xacro (robot description, xacro)
@@ -76,5 +76,14 @@
     mass="${wheel_mass}"
   />
-  <link name="front_rs_depth_optical_frame">
+  <!-- IsaacSim will likely not respect joint angles for realsense joints -->
+  <joint
+    name="base_link_to_front_rs" type="fixed">
+    <origin
+      xyz="0.410335 0 0.0892"
+      rpy="-1.57 1.57 0" />
+    <parent link="base_link" />
+    <child link="front_rs_depth_optical_frame" />
+  </joint>
+  <link name="rear_rs_depth_optical_frame">
     <inertial>
       <mass value="0.025" />
@@ -91,11 +100,60 @@
     </collision>
   </link>
+  <!-- IsaacSim will likely not respect joint angles for realsense joints -->
   <joint
-    name="base_link_to_front_rs" type="fixed">
+    name="base_link_to_rear_rs" type="fixed">
     <origin
-      xyz="0 0 0"
-      rpy="0 0 0" />
+      xyz="-0.41 0 0.089"
+      rpy="-1.57 -1.57 0" />
     <parent link="base_link" />
-    <child link="front_rs_depth_optical_frame" />
+    <child link="rear_rs_depth_optical_frame" />
+  </joint>
+  <link name="left_rs_depth_optical_frame">
+    <inertial>
+      <mass value="0.025" />
+    </inertial>
+    <visual>
+      <origin
+        xyz="0 0 0"
+        rpy="0 0 0" />
+    </visual>
+    <collision>
+      <origin
+        xyz="0 0 0"
+        rpy="0 0 0" />
+    </collision>
+  </link>
+  <!-- IsaacSim will likely not respect joint angles for realsense joints -->
+  <joint
+    name="base_link_to_left_rs" type="fixed">
+    <origin
+      xyz="0 0.247 0.089"
+      rpy="-1.57 0 0" />
+    <parent link="base_link" />
+    <child link="left_rs_depth_optical_frame" />
+  </joint>
+  <link name="right_rs_depth_optical_frame">
+    <inertial>
+      <mass value="0.025" />
+    </inertial>
+    <visual>
+      <origin
+        xyz="0 0 0"
+        rpy="0 0 0" />
+    </visual>
+    <collision>
+      <origin
+        xyz="0 0 0"
+        rpy="0 0 0" />
+    </collision>
+  </link>
+  <!-- IsaacSim will likely not respect joint angles for realsense joints -->
+  <joint
+    name="base_link_to_right_rs" type="fixed">
+    <origin
+      xyz="0 -0.247 0.089"
+      rpy="1.57 0 3.14" />
+    <parent link="base_link" />
+    <child link="right_rs_depth_optical_frame" />
   </joint>
 </robot>
