Commit message: Added more realistic pipe rail, to be used for SLAMing greenhouse

File: simulation/isaacsim/models/rails/rails.urdf (robot description, URDF)
Before this commit: robot rails, 2 links, 1 joints
Links:
- removed link rail1
- removed link rail2
- added link base_link
- added link end_rail_1; visual cylinder length=0.39 radius=0.03
- added link end_rail_2; visual cylinder length=0.39 radius=0.03
- added link fillet_1; visual cylinder length=0.06 radius=0.12
- added link fillet_2; visual cylinder length=0.06 radius=0.12
- added link fillet_3; visual cylinder length=0.06 radius=0.12
- added link fillet_4; visual cylinder length=0.06 radius=0.12
- added link rail_1; visual cylinder length=21.76 radius=0.03
- added link rail_2; visual cylinder length=21.76 radius=0.03
Joints:
- removed joint rails_joint
- added joint base_link_to_end_rail_1: type fixed, parent base_link, child end_rail_1, origin xyz=-11 0 0 rpy=1.57 0 0
- added joint base_link_to_end_rail_2: type fixed, parent base_link, child end_rail_2, origin xyz=11 0 0 rpy=1.57 0 0
- added joint base_link_to_fillet_1: type fixed, parent base_link, child fillet_1, origin xyz=-10.91 -0.21 0 rpy=0 0 0
- added joint base_link_to_fillet_2: type fixed, parent base_link, child fillet_2, origin xyz=-10.91 0.21 0 rpy=0 0 0
- added joint base_link_to_fillet_3: type fixed, parent base_link, child fillet_3, origin xyz=10.91 -0.21 0 rpy=0 0 0
- added joint base_link_to_fillet_4: type fixed, parent base_link, child fillet_4, origin xyz=10.91 0.21 0 rpy=0 0 0
- added joint base_link_to_rail_1: type fixed, parent base_link, child rail_1, origin xyz=0 0.3 0 rpy=0 1.57 0
- added joint base_link_to_rail_2: type fixed, parent base_link, child rail_2, origin xyz=0.0 -0.3 0 rpy=0 1.57 0

Commit message: Added new pipe rails and plants to sim, with a bit of variance in positioning

File: simulation/isaacsim/models/rails/rails.urdf (robot description, URDF)
Before this commit: robot greenhouse_piperail, 9 links, 8 joints
Links:
- link end_rail_1: geometry collision cylinder length=0.39 radius=0.03; visual cylinder length=0.39 radius=0.03
- link end_rail_2: geometry collision cylinder length=0.39 radius=0.03; visual cylinder length=0.39 radius=0.03
- link fillet_1: geometry collision cylinder length=0.06 radius=0.12; visual cylinder length=0.06 radius=0.12
- link fillet_2: geometry collision cylinder length=0.06 radius=0.12; visual cylinder length=0.06 radius=0.12
- link fillet_3: geometry collision cylinder length=0.06 radius=0.12; visual cylinder length=0.06 radius=0.12
- link fillet_4: geometry collision cylinder length=0.06 radius=0.12; visual cylinder length=0.06 radius=0.12
- link rail_1: geometry collision cylinder length=21.76 radius=0.03; visual cylinder length=21.76 radius=0.03
- link rail_2: geometry collision cylinder length=21.76 radius=0.03; visual cylinder length=21.76 radius=0.03
